File: hardware/Source/Ver_1.0.0/Automative_Hexapod.kicad_sch (KiCad schematic)
At the start: 70 parts, among them J1 MPU6050, J2 Conn_01x04_Pin, J3 Conn_01x04_Pin, J4 Conn_01x04_Pin, J5 Conn_01x03_Pin, Q1 LN2302LT1G, Q2 LN2302LT1G, Q3 LN2302LT1G, Q4 LN2302LT1G, Q5 LN2302LT1G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

Commit message: update folder hardware
Other:
- title: (none) -> MAIN
