File: hardware/Source/Ver_1.0.0/Automative_Hexapod.kicad_sch (KiCad schematic)
At the start: 70 parts, among them J1 MPU6050, J2 Conn_01x04_Pin, J3 Conn_01x04_Pin, J4 Conn_01x04_Pin, J5 Conn_01x03_Pin, Q1 LN2302LT1G, Q2 LN2302LT1G, Q3 LN2302LT1G, Q4 LN2302LT1G, Q5 LN2302LT1G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

Commit message: Update Library for Ver 2
Parts:
- C1, C12, C13, C14, C19, C20, C21, C22, C27, C28, C3, C31, C37, C5, C7, C9: Supply Name (none) -> Thegioiic; Supply Part Number (none) -> Tụ Gốm 0805 10uF 16V; Supply name Thegioiic -> (none); Supply part number Tụ Gốm 0805 10uF 16V -> (none)
- C10, C11, C15, C16, C17, C18, C2, C23, C24, C25, C26, C30, C39, C4, C6, C8: Supply Name (none) -> Thegioiic; Supply Part Number (none) -> Tụ Gốm 0805 100nF (0.1uF) 50V; Supply name Thegioiic -> (none); Supply part number Tụ Gốm 0805 100nF (0.1uF) 50V -> (none)
- C29: Supply Name (none) -> Thegioiic; Supply Part Number (none) -> Tụ Nhôm SMD 330uF 50V 10x10.5mm; Supply name Thegioiic -> (none); Supply part number Tụ Nhôm SMD 330uF 50V 10x10.5mm -> (none)
- C38: Supply Name (none) -> Thegioiic; Supply Part Number (none) -> Tụ Nhôm SMD 220uF 50V 10x10.5mm; Supply name Thegioiic -> (none); Supply part number Tụ Nhôm SMD 220uF 50V 10x10.5mm -> (none)
- C45, C46: Supply Name (none) -> Thegioiic; Supply Part Number (none) -> Tụ Gốm 0805 1uF 16V; Supply name Thegioiic -> (none); Supply part number Tụ Gốm 0805 1uF 16V -> (none)
- D1: Supply Name (none) -> Thegioiic; Supply Part Number (none) -> LED Xanh Lá 0805 Dán SMD Trong Suốt; Supply name Thegioiic -> (none); Supply part number LED Xanh Lá 0805 Dán SMD Trong Suốt -> (none)
- J2, J3, J4: footprint automative_hexapod:PinHeader_1x04_P2.54mm_Vertical -> automative_hexapod:PinHeader_1x04_P1.00mm_Vertical
- J5: footprint automative_hexapod:PinHeader_1x03_P2.54mm_Vertical -> automative_hexapod:PinHeader_1x03_P1.00mm_Vertical
- Q1, Q2, Q3, Q4, Q5, Q6, Q9: Supply Name (none) -> Thegioiic; Supply Part Number (none) -> LN2302LT1G MOSFET Kênh N 20V 2.3A SOT-23-3; Supply name Thegioiic -> (none); Supply part number LN2302LT1G MOSFET Kênh N 20V 2.3A SOT-23-3 -> (none)
- R1, R10, R11, R12, R17, R19, R2, R3, R4, R5, R6, R7, R8, R9: Supply Name (none) -> thegioiic; Supply Part Number (none) -> Điện Trở 10 KOhm 0805 1%; Supply name thegioiic -> (none); Supply part number Điện Trở 10 KOhm 0805 1% -> (none)
- R13: Supply Name (none) -> thegioiic; Supply Part Number (none) -> Điện Trở 10.5 KOhm 0805 1%; Supply name thegioiic -> (none); Supply part number Điện Trở 10.5 KOhm 0805 1% -> (none)
- R14: Supply Name (none) -> thegioiic; Supply Part Number (none) -> Điện Trở 2 KOhm 0805 1%; Supply name thegioiic -> (none); Supply part number Điện Trở 2 KOhm 0805 1% -> (none)
- R18: Supply Name (none) -> thegioiic; Supply Part Number (none) -> Điện Trở 1 KOhm 0805 1%; Supply name thegioiic -> (none); Supply part number Điện Trở 1 KOhm 0805 1% -> (none)
