File: hardware/Source/Ver_1.0.0/Automative_Hexapod.kicad_sch (KiCad schematic)
At the start: 70 parts, among them J1 MPU6050, J2 Conn_01x04_Pin, J3 Conn_01x04_Pin, J4 Conn_01x04_Pin, J5 Conn_01x03_Pin, Q1 LN2302LT1G, Q2 LN2302LT1G, Q3 LN2302LT1G, Q4 LN2302LT1G, Q5 LN2302LT1G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

Commit message: update pcb v1.1.0
Parts:
- C1, C12, C13, C14, C19, C20, C21, C22, C27, C28, C3, C31, C37, C5, C7, C9: Supply Name (none) -> Thegioiic; Supply Part Number (none) -> Tụ Gốm 0805 10uF 16V; Supply URL https://www.thegioiic.com/tu-gom-0805-10uf-16v -> https://www.Thegioiic.com/tu-gom-0805-10uf-16v; Supply name Thegioiic -> (none); Supply part number Tụ Gốm 0805 10uF 16V -> (none)
- C10, C11, C15, C16, C17, C18, C2, C23, C24, C25, C26, C30, C39, C4, C6, C8: Supply Name (none) -> Thegioiic; Supply Part Number (none) -> Tụ Gốm 0805 100nF (0.1uF) 50V; Supply URL https://www.thegioiic.com/tu-gom-0805-100nf-0-1uf-50v -> https://www.Thegioiic.com/tu-gom-0805-100nf-0-1uf-50v; Supply name Thegioiic -> (none); Supply part number Tụ Gốm 0805 100nF (0.1uF) 50V -> (none)
- C29: Supply Name (none) -> Thegioiic; Supply Part Number (none) -> Tụ Nhôm SMD 330uF 50V 10x10.5mm; Supply URL https://www.thegioiic.com/tu-nhom-smd-330uf-50v-10x10-5mm -> https://www.Thegioiic.com/tu-nhom-smd-330uf-50v-10x10-5mm; Supply name Thegioiic -> (none); Supply part number Tụ Nhôm SMD 330uF 50V 10x10.5mm -> (none)
- C38: Supply Name (none) -> Thegioiic; Supply Part Number (none) -> Tụ Nhôm SMD 220uF 50V 10x10.5mm; Supply URL https://www.thegioiic.com/tu-nhom-smd-220uf-50v-10x10-5mm -> https://www.Thegioiic.com/tu-nhom-smd-220uf-50v-10x10-5mm; Supply name Thegioiic -> (none); Supply part number Tụ Nhôm SMD 220uF 50V 10x10.5mm -> (none)
- C45, C46: Supply Name (none) -> Thegioiic; Supply Part Number (none) -> Tụ Gốm 0805 1uF 16V; Supply URL https://www.thegioiic.com/tu-gom-0805-1uf-16v -> https://www.Thegioiic.com/tu-gom-0805-1uf-16v; Supply name Thegioiic -> (none); Supply part number Tụ Gốm 0805 1uF 16V -> (none)
- D1: Supply Name (none) -> Thegioiic; Supply Part Number (none) -> LED Xanh Lá 0805 Dán SMD Trong Suốt; Supply URL https://www.thegioiic.com/led-xanh-la-0805-dan-smd-trong-su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 -> https://www.Thegioiic.com/led-xanh-la-0805-dan-smd-trong-su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; Supply name Thegioiic -> (none); Supply part number LED Xanh Lá 0805 Dán SMD Trong Suốt -> (none)
- D2: Supply URL https://www.thegioiic.com/mbr20100ct-diode-schottky-100v-10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 -> https://www.Thegioiic.com/mbr20100ct-diode-schottky-100v-10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
- J1: Supply URL https://www.thegioiic.com/hang-rao-duc-don-2-54mm-40-chan-1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 -> https://www.Thegioiic.com/hang-rao-duc-don-2-54mm-40-chan-1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
- J2, J3, J4: footprint automative_hexapod:PinHeader_1x04_P2.54mm_Vertical -> automative_hexapod:PinHeader_1x04_P1.00mm_Vertical; Supply URL https://www.thegioiic.com/hang-rao-duc-don-2-54mm-40-chan-1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 -> https://www.Thegioiic.com/hang-rao-duc-don-2-54mm-40-chan-1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
- J5: footprint automative_hexapod:PinHeader_1x03_P2.54mm_Vertical -> automative_hexapod:PinHeader_1x03_P1.00mm_Vertical; Supply URL https://www.thegioiic.com/hang-rao-duc-don-2-54mm-40-chan-1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 -> https://www.Thegioiic.com/hang-rao-duc-don-2-54mm-40-chan-1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
- L1: Supply Name ThegioiIC -> Thegioiic; Supply URL https://www.thegioiic.com/cuon-cam-dan-smd-cdrh127-1280-270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 -> https://www.Thegioiic.com/cuon-cam-dan-smd-cdrh127-1280-270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
- Q1, Q2, Q3, Q4, Q5, Q6, Q9: Supply Name (none) -> Thegioiic; Supply Part Number (none) -> LN2302LT1G MOSFET Kênh N 20V 2.3A SOT-23-3; Supply URL https://www.thegioiic.com/ln2302lt1g-mosfet-kenh-n-20v-2-3a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 -> https://www.Thegioiic.com/ln2302lt1g-mosfet-kenh-n-20v-2-3a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; Supply name Thegioiic -> (none); Supply part number LN2302LT1G MOSFET Kênh N 20V 2.3A SOT-23-3 -> (none)
- R1, R10, R11, R12, R17, R19, R2, R3, R4, R5, R6, R7, R8, R9: Supply Name (none) -> Thegioiic; Supply Part Number (none) -> Điện Trở 10 KOhm 0805 1%; Supply URL https://www.thegioiic.com/dien-tro-10-kohm-0805-1- -> https://www.Thegioiic.com/dien-tro-10-kohm-0805-1-; Supply name thegioiic -> (none); Supply part number Điện Trở 10 KOhm 0805 1% -> (none)
- R13: Supply Name (none) -> Thegioiic; Supply Part Number (none) -> Điện Trở 10.5 KOhm 0805 1%; Supply URL https://www.thegioiic.com/dien-tro-10-5-kohm-0805-1- -> https://www.Thegioiic.com/dien-tro-10-5-kohm-0805-1-; Supply name thegioiic -> (none); Supply part number Điện Trở 10.5 KOhm 0805 1% -> (none)
- R14: Supply Name (none) -> Thegioiic; Supply Part Number (none) -> Điện Trở 2 KOhm 0805 1%; Supply URL https://www.thegioiic.com/dien-tro-2-kohm-0805-1- -> https://www.Thegioiic.com/dien-tro-2-kohm-0805-1-; Supply name thegioiic -> (none); Supply part number Điện Trở 2 KOhm 0805 1% -> (none)
- R18: Supply Name (none) -> Thegioiic; Supply Part Number (none) -> Điện Trở 1 KOhm 0805 1%; Supply URL https://www.thegioiic.com/dien-tro-1-kohm-0805-1- -> https://www.Thegioiic.com/dien-tro-1-kohm-0805-1-; Supply name thegioiic -> (none); Supply part number Điện Trở 1 KOhm 0805 1% -> (none)
- U2: Supply URL https://www.thegioiic.com/xl4005e1-ic-dieu-chinh-giam-ap-5a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 -> https://www.Thegioiic.com/xl4005e1-ic-dieu-chinh-giam-ap-5a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
