File: hardware/Source/Automative_Hexapod/Automative_Hexapod.kicad_pcb (KiCad board)
At the start: 2 copper layers, 70 parts, among them J1 Conn_02x02, J2 Conn_02x02, J3 Conn_02x02, J4 Conn_02x02, J6 Conn_02x02, Q1 LN2302LT1G, Q2 LN2302LT1G, Q3 LN2302LT1G, Q4 LN2302LT1G, Q5 LN2302LT1G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

Commit message: upload pcb
Parts:
- moved D1 63.5 mm to (222.4, 80.1)
- moved R11 63.5 mm to (229.4, 104.3)
- moved R5 63.5 mm to (225.3, 104.3)
- moved Q1 63.5 mm to (207.9, 85.4)
- moved Q2 63.5 mm to (212.6, 85.4)
- moved Q3 63.5 mm to (217.2, 85.4)
- moved Q4 63.5 mm to (221.9, 85.4)
- moved Q5 63.5 mm to (207.9, 90.3)
- moved Q6 63.5 mm to (212.6, 90.3)
- moved Q9 63.5 mm to (217.2, 90.3)
- moved R1 63.5 mm to (225.3, 94.0)
- moved R10 63.5 mm to (229.4, 101.8)
- moved R12 63.5 mm to (229.4, 106.9)
- moved R17 63.5 mm to (233.4, 94.0)
- moved R18 63.5 mm to (233.4, 96.6)
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Other:
- board outline added: 100 x 100 mm

Commit message: Update PCB: TestBoard_V1.0.0
Parts:
- removed C41: 10uF/16V, automative_hexapod:Ceramic_Cap_0805
- removed C43: 100nF/50V, automative_hexapod:Ceramic_Cap_0805
- removed J6: Conn_02x02, automative_hexapod:PinHeader_2x02_P2.54mm_Vertical_SMD
- removed R20: 16K/1%/1/8W, automative_hexapod:Res_0805
- removed R21: 3K/1%/1/8W, automative_hexapod:Res_0805
- added C30: 100nF/50V, automative_hexapod:Ceramic_Cap_0805, F.Cu at (175.8, 133.2)
- added C31: 10uF/16V, automative_hexapod:Ceramic_Cap_0805, F.Cu at (175.8, 135.6)
- added J5: Conn_01x03_Pin, automative_hexapod:PinHeader_1x03_P1.00mm_Vertical, B.Cu at (172.2, 131.1)
- added R13: 10.5K/1%/1/8W, automative_hexapod:Res_0805, F.Cu at (192.2, 110.4)
- added R14: 2K/1%/1/8W, automative_hexapod:Res_0805, F.Cu at (196.2, 110.4)
- C11, C17, C18, C25, C26: value 10uF/16V -> 100nF/50V
- C12, C19, C20, C27, C28: value 100nF/50V -> 10uF/16V
- D2: moved to B.Cu
- J1: value Conn_02x02 -> MPU6050; footprint automative_hexapod:PinHeader_2x02_P2.54mm_Vertical_SMD -> automative_hexapod:MPU6050; moved to B.Cu
- J2, J3, J4: value Conn_02x02 -> Conn_01x04_Pin; footprint automative_hexapod:PinHeader_2x02_P2.54mm_Vertical_SMD -> automative_hexapod:PinHeader_1x04_P1.00mm_Vertical; moved to B.Cu
- moved C20 143.8 mm to (119.1, 136.3), turned to 180 degrees
- moved C19 136.2 mm to (119.1, 120.8), turned to 180 degrees
- moved C14 131.7 mm to (123.3, 136.4)
- moved C28 131.2 mm to (119.4, 104.4), turned to 180 degrees
- moved C18 126.9 mm to (119.1, 133.9), turned to 180 degrees
- moved C16 126.7 mm to (123.3, 134.0)
- moved J2 125.8 mm to (115.5, 131.6)
- moved C13 124.1 mm to (123.3, 120.9)
- moved C17 120.5 mm to (119.1, 118.4), turned to 180 degrees
- moved C15 119.7 mm to (123.3, 118.5)
- moved C22 119.4 mm to (123.7, 104.5)
- moved C26 117.9 mm to (119.4, 101.9), turned to 180 degrees
- moved R8 116.4 mm to (118.0, 130.7), turned to -90 degrees
- moved C24 116.0 mm to (123.7, 102.0)
- moved C21 115.8 mm to (123.7, 93.0)
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Connections:
- J1 pad 1: MPU6050_I2C_SCL -> +5V
- J1 pad 2: +5V -> GND
- J1 pad 3: MPU6050_I2C_SDA -> MPU6050_I2C_SCL
- J1 pad 4: GND -> MPU6050_I2C_SDA
- J2 pad 1: PCA9685_I2C_SCL -> +5V
- J2 pad 2: +5V -> GND
- J2 pad 3: PCA9685_I2C_SDA -> PCA9685_I2C_SCL
- J2 pad 4: GND -> PCA9685_I2C_SDA
- J3 pad 1: PCA9685_I2C_SCL -> +5V
- J3 pad 2: +5V -> GND
- J3 pad 4: GND -> PCA9685_I2C_SCL
- J4 pad 1: HCSR04_TRIG -> +5V
- J4 pad 2: +5V -> GND
- J4 pad 4: GND -> HCSR04_TRIG
- Q3 pad 2: BBAI_I2C_SCL -> BBAI_I2C_SDA
- Q3 pad 3: PCA9685_I2C_SCL -> PCA9685_I2C_SDA
- Q4 pad 2: BBAI_I2C_SDA -> BBAI_I2C_SCL
- Q4 pad 3: PCA9685_I2C_SDA -> PCA9685_I2C_SCL
- R5 pad 1: BBAI_I2C_SCL -> BBAI_I2C_SDA
- R6 pad 1: BBAI_I2C_SDA -> BBAI_I2C_SCL
- R7 pad 1: PCA9685_I2C_SCL -> PCA9685_I2C_SDA
- R8 pad 1: PCA9685_I2C_SDA -> PCA9685_I2C_SCL
- U1 pad P8_1: unconnected-(U1-GND-PadP8_1) -> GND
- U1 pad P8_2: unconnected-(U1-GND-PadP8_2) -> GND
Routing:
- net GND: track 77.5 -> 615.1 mm, vias 0 -> 18
- net +3.3V: track 0.00 -> 351.4 mm, vias 0 -> 14
- net +5V: track 12.7 -> 351.3 mm, vias 0 -> 13
- net BBAI_I2C_SDA: track 0.00 -> 100.7 mm
- net BBAI_PWM1A: track 0.00 -> 93.9 mm
- net BBAI_I2C_SCL: track 0.00 -> 69.8 mm
- net PCA9685_I2C_SCL: track 0.00 -> 26.7 mm
- net PCA9685_I2C_SDA: track 0.00 -> 23.7 mm
- net BBAI_ECHO: track 0.00 -> 19.4 mm
- net HCSR04_TRIG: track 0.00 -> 15.4 mm
- net BBAI_TRIG: track 0.00 -> 14.7 mm
- net MPU6050_I2C_SDA: track 0.00 -> 10.4 mm
- net Net-(U2-FB): track 3.37 -> 12.0 mm
- net VCC: track 14.0 -> 22.3 mm, vias 0 -> 1
- net MPU6050_I2C_SCL: track 0.00 -> 6.17 mm
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- added copper zone on F.Cu, net +5V
- added copper zone on F.Cu, net VCC
Other:
- board size 100 x 100 mm -> 110.1 x 111.8 mm

Commit message: Pull request
Parts:
- J2, J3, J4: footprint automative_hexapod:PinHeader_1x04_P1.00mm_Vertical -> automative_hexapod:PinHeader_1x04_P2.54mm_Vertical
- J5: footprint automative_hexapod:PinHeader_1x03_P1.00mm_Vertical -> automative_hexapod:PinHeader_1x03_P2.54mm_Vertical
- moved R17 70.5 mm to (111.3, 121.1), turned to 0 degrees
- moved Q9 66.9 mm to (111.3, 124.4), turned to 180 degrees
- moved C39 66.5 mm to (114.6, 122.2), turned to 90 degrees
- moved C37 64.6 mm to (117.0, 122.2), turned to 90 degrees
- moved J4 63.6 mm to (53.6, 87.4)
- moved R19 63.5 mm to (111.3, 127.6), turned to 0 degrees
- moved C12 61.7 mm to (103.4, 126.4)
- moved C5 61.7 mm to (84.6, 121.1)
- moved C6 61.7 mm to (84.6, 123.4)
- moved C7 61.7 mm to (88.9, 121.2)
- moved C8 61.7 mm to (88.9, 123.6)
- moved Q2 61.7 mm to (97.8, 124.2)
- moved C13 61.7 mm to (62.1, 112.9)
- moved C15 61.7 mm to (62.1, 110.5)
- moved C26 61.7 mm to (58.2, 93.9)
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Routing:
- net +3.3V: track 351.4 -> 369.4 mm
- net HCSR04_ECHO: track 5.31 -> 18.4 mm
- net GND: track 615.1 -> 625.0 mm, vias 18 -> 19
- net HCSR04_TRIG: track 15.4 -> 6.96 mm
- net BBAI_PWM1A: track 93.9 -> 86.7 mm
- net +5V: track 351.3 -> 355.1 mm, vias 13 -> 9
- net PCA9685_I2C_SCL: track 26.7 -> 28.3 mm
- net PCA9685_I2C_SDA: track 23.7 -> 22.4 mm
- net FAN_PWM1A: track 5.43 -> 6.63 mm
