File: hardware/Source/Automative_Hexapod/Automative_Hexapod.kicad_sch (KiCad schematic)
At the start: 70 parts, among them J1 Conn_02x02, J2 Conn_02x02, J3 Conn_02x02, J4 Conn_02x02, J6 Conn_02x02, Q1 LN2302LT1G, Q2 LN2302LT1G, Q3 LN2302LT1G, Q4 LN2302LT1G, Q5 LN2302LT1G, Q6 LN2302LT1G, Q9 LN2302LT1G, U2 XL4005E1

Commit message: Update PCB: TestBoard_V1.0.0
Parts:
- removed C11, C17, C18, C25, C26, C41: 10uF/16V, automative_hexapod:Ceramic_Cap_0805, symbol automative_hexapod:Ceramic_Cap_0805_10uF_16V
- removed C12, C19, C20, C27, C28, C43: 100nF/50V, automative_hexapod:Ceramic_Cap_0805, symbol automative_hexapod:Ceramic_Cap_0805_100nF_50V
- removed J1, J2, J3, J4, J6: Conn_02x02, automative_hexapod:PinHeader_2x02_P2.54mm_Vertical_SMD, symbol automative_hexapod:Conn_02x02
- removed R20: 16K/1%/1/8W, automative_hexapod:Res_0805, symbol automative_hexapod:Res_16K_0805_1%
- removed R21: 3K/1%/1/8W, automative_hexapod:Res_0805, symbol automative_hexapod:Res_3K_0805_1%
- added C11, C17, C18, C25, C26, C30: 100nF/50V, automative_hexapod:Ceramic_Cap_0805, symbol automative_hexapod:Ceramic_Cap_0805_100nF_50V
- added C12, C19, C20, C27, C28, C31: 10uF/16V, automative_hexapod:Ceramic_Cap_0805, symbol automative_hexapod:Ceramic_Cap_0805_10uF_16V
- added J1: MPU6050, automative_hexapod:MPU6050, symbol automative_hexapod:MPU6050
- added J2, J3, J4: Conn_01x04_Pin, automative_hexapod:PinHeader_1x04_P1.00mm_Vertical, symbol automative_hexapod:Conn_01x04_Pin
- added J5: Conn_01x03_Pin, automative_hexapod:PinHeader_1x03_P1.00mm_Vertical, symbol automative_hexapod:Conn_01x03_Pin
- added R13: 10.5K/1%/1/8W, automative_hexapod:Res_0805, symbol automative_hexapod:Res_10.5K_0805_1%
- added R14: 2K/1%/1/8W, automative_hexapod:Res_0805, symbol automative_hexapod:Res_2K_0805_1%
Connections:
- net +5V: now also C11.2, C12.2, C17.2, C18.2, C19.2, C20.2, C25.2, C26.2, C27.2, C28.2, C30.2, C31.2, J1.1 (Pin_1), J2.1 (Pin_1), J3.1 (Pin_1), J4.1 (Pin_1), J5.1 (Pin_1), R13.2
- net BBAI_I2C_SCL: now also Q4.2 (S), R6.1; no longer Q3.2 (S), R5.1
- net BBAI_I2C_SDA: now also Q3.2 (S), R5.1; no longer Q4.2 (S), R6.1
- net FAN_PWM1A: now also J5.3 (Pin_3)
- net GND: now also U1.P8_1 (GND), U1.P8_2 (GND), C11.1, C12.1, C17.1, C18.1, C19.1, C20.1, C25.1, C26.1, C27.1, C28.1, C30.1, C31.1, J1.2 (Pin_2), J2.2 (Pin_2), J3.2 (Pin_2), J4.2 (Pin_2), J5.2 (Pin_2), R14.1
- net HCSR04_ECHO: now also J4.3 (Pin_3)
- net HCSR04_TRIG: now also J4.4 (Pin_4)
- net MPU6050_I2C_SCL: now also J1.3 (Pin_3)
- net MPU6050_I2C_SDA: now also J1.4 (Pin_4)
- net PCA9685_I2C_SCL: now also Q4.3 (D), R8.1, J2.3 (Pin_3), J3.4 (Pin_4); no longer Q3.3 (D), R7.1
- net PCA9685_I2C_SDA: now also Q3.3 (D), R7.1, J2.4 (Pin_4), J3.3 (Pin_3); no longer Q4.3 (D), R8.1
- net at U2.2 (FB): now also R13.1, R14.2
- no-connect marks 82 -> 83
Other:
- note added: "Thermal Fan"
- note removed: "FAN"
- note removed: "JACK LIPO"
- moved on the sheet: C7, C8

Commit message: Pull request
Parts:
- J2, J3, J4: footprint automative_hexapod:PinHeader_1x04_P1.00mm_Vertical -> automative_hexapod:PinHeader_1x04_P2.54mm_Vertical
- J5: footprint automative_hexapod:PinHeader_1x03_P1.00mm_Vertical -> automative_hexapod:PinHeader_1x03_P2.54mm_Vertical
Changed lines of the file:
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@@
 			)
 		)
-		(property "Footprint" "automative_hexapod:PinHeader_1x04_P1.00mm_Vertical"
+		(property "Footprint" "automative_hexapod:PinHeader_1x04_P2.54mm_Vertical"
 			(at 208.28 114.3 0)
 			(effects
@@
 	)
 	(symbol
-		(lib_name "Cap_Polarized_SMD_220uF_50V_1")
 		(lib_id "automative_hexapod:Cap_Polarized_SMD_220uF_50V")
 		(at 33.02 187.96 270)
@@
 			)
 		)
-		(property "Footprint" "automative_hexapod:PinHeader_1x04_P1.00mm_Vertical"
+		(property "Footprint" "automative_hexapod:PinHeader_1x04_P2.54mm_Vertical"
 			(at 259.08 139.7 0)
 			(effects
@@
 			)
 		)
-		(property "Footprint" "automative_hexapod:PinHeader_1x03_P1.00mm_Vertical"
+		(property "Footprint" "automative_hexapod:PinHeader_1x03_P2.54mm_Vertical"
 			(at 209.55 139.7 0)
 			(effects
@@
 			)
 		)
-		(property "Footprint" "automative_hexapod:PinHeader_1x04_P1.00mm_Vertical"
+		(property "Footprint" "automative_hexapod:PinHeader_1x04_P2.54mm_Vertical"
 			(at 259.08 160.02 0)
 			(effects
