File: hardware/Source/Ver_1.1.0/Automative_Hexapod.kicad_pcb (KiCad board)
At the start: 2 copper layers, 110.1 x 111.8 mm, 70 parts, among them J1 MPU6050, J2 Conn_01x04_Pin, J3 Conn_01x04_Pin, J4 Conn_01x04_Pin, J5 Conn_01x03_Pin, Q1 LN2302LT1G, Q2 LN2302LT1G, Q3 LN2302LT1G, Q4 LN2302LT1G, Q5 LN2302LT1G, Q6 LN2302LT1G, Q9 LN2302LT1G, U2 XL4005E1

Commit message: Update Library for Ver 2
Parts:
- removed J5: Conn_01x03_Pin, automative_hexapod:PinHeader_1x03_P2.54mm_Vertical
- removed Q6, Q9: LN2302LT1G, automative_hexapod:SOT23
- added C32: 100nF, automative_hexapod:Ceramic_Cap_0805, B.Cu at (231.8, 61.0)
- added C33: 10uF, automative_hexapod:Ceramic_Cap_0805, B.Cu at (221.6, 51.5)
- added C34: 100nF, automative_hexapod:Ceramic_Cap_0805, B.Cu at (221.6, 54.2)
- added C35: 10uF, automative_hexapod:Ceramic_Cap_0805, B.Cu at (215.2, 81.3)
- added C36: 10uF, automative_hexapod:Ceramic_Cap_0805, B.Cu at (215.2, 84.0)
- added C40: 10uF, automative_hexapod:Ceramic_Cap_0805, B.Cu at (215.2, 94.9)
- added C41: 100nF, automative_hexapod:Ceramic_Cap_0805, B.Cu at (215.2, 97.6)
- added C42: 100nF, automative_hexapod:Ceramic_Cap_0805, B.Cu at (215.2, 100.3)
- added C43: 100nF, automative_hexapod:Ceramic_Cap_0805, B.Cu at (215.2, 103.0)
- added C44: 100nF, automative_hexapod:Ceramic_Cap_0805, B.Cu at (211.2, 81.3)
- added C47: 10uF, automative_hexapod:Ceramic_Cap_0805, B.Cu at (211.2, 89.4)
- added C48: 10uF, automative_hexapod:Ceramic_Cap_0805, B.Cu at (211.2, 92.2)
- added C49: 10uF, automative_hexapod:Ceramic_Cap_0805, B.Cu at (211.2, 94.9)
- added C50: 10uF, automative_hexapod:Ceramic_Cap_0805, B.Cu at (211.2, 97.6)
- added C51: 10uF, automative_hexapod:Ceramic_Cap_0805, B.Cu at (211.2, 100.3)
- added C52: 10uF, automative_hexapod:Ceramic_Cap_0805, B.Cu at (211.2, 103.0)
- added C53: 100nF, automative_hexapod:Ceramic_Cap_0805, B.Cu at (207.1, 81.3)
- added C54: 100nF, automative_hexapod:Ceramic_Cap_0805, B.Cu at (207.1, 84.0)
- added C55: 100nF, automative_hexapod:Ceramic_Cap_0805, B.Cu at (207.1, 86.7)
- added C56: 100nF, automative_hexapod:Ceramic_Cap_0805, B.Cu at (207.1, 89.4)
- added C57: 100nF, automative_hexapod:Ceramic_Cap_0805, B.Cu at (207.1, 92.2)
- added C58: 100nF, automative_hexapod:Ceramic_Cap_0805, B.Cu at (207.1, 94.9)
- added C59: 10uF, automative_hexapod:Ceramic_Cap_0805, B.Cu at (207.1, 97.6)
- added C60: 10uF, automative_hexapod:Ceramic_Cap_0805, B.Cu at (207.1, 100.3)
- added C61: 10uF, automative_hexapod:Ceramic_Cap_0805, B.Cu at (207.1, 103.0)
- added C62: 10uF, automative_hexapod:Ceramic_Cap_0805, B.Cu at (203.1, 81.3)
- added C63: 10uF, automative_hexapod:Ceramic_Cap_0805, B.Cu at (203.1, 84.0)
- added C64: 100nF, automative_hexapod:Ceramic_Cap_0805, B.Cu at (203.1, 86.7)
- added C65: 100nF, automative_hexapod:Ceramic_Cap_0805, B.Cu at (203.1, 89.4)
- added C66: 100nF, automative_hexapod:Ceramic_Cap_0805, B.Cu at (203.1, 92.2)
- added C67: 100nF, automative_hexapod:Ceramic_Cap_0805, B.Cu at (203.1, 94.9)
- added C68: 100nF, automative_hexapod:Ceramic_Cap_0805, B.Cu at (203.1, 97.6)
- added C69: 10uF, automative_hexapod:Ceramic_Cap_0805, B.Cu at (203.1, 100.3)
- added C70: 10uF, automative_hexapod:Ceramic_Cap_0805, B.Cu at (203.1, 103.0)
- added C71: 10uF, automative_hexapod:Ceramic_Cap_0805, B.Cu at (199.0, 81.3)
- added C72: 10uF, automative_hexapod:Ceramic_Cap_0805, B.Cu at (199.0, 84.0)
- added C73: 10uF, automative_hexapod:Ceramic_Cap_0805, B.Cu at (199.0, 86.7)
- added C74: 100nF, automative_hexapod:Ceramic_Cap_0805, B.Cu at (199.0, 89.4)
- added C75: 100nF, automative_hexapod:Ceramic_Cap_0805, B.Cu at (199.0, 92.2)
- added C76: 100nF, automative_hexapod:Ceramic_Cap_0805, B.Cu at (199.0, 94.9)
- added C77: 100nF, automative_hexapod:Ceramic_Cap_0805, B.Cu at (199.0, 97.6)
- added C78: 100nF, automative_hexapod:Ceramic_Cap_0805, B.Cu at (199.0, 100.3)
- added D3: 3.3V, automative_hexapod:LED_0805, B.Cu at (258.9, 45.9)
- added D4: MBR20100CT, automative_hexapod:TO-220-3, B.Cu at (258.0, 36.3)
- added D5: LED_0805, automative_hexapod:LED_0805, B.Cu at (238.0, 57.1)
- added F1: Fuse, automative_hexapod:FUSE_SMD_1808, B.Cu at (190.3, 146.0)
- added J10: Connector, automative_hexapod:JST-XH-SMD-3-2.54mm, B.Cu at (224.2, 119.8)
- added J11: Connector, automative_hexapod:JST-XH-SMD-3-2.54mm, B.Cu at (266.4, 119.4)
- added J12: Connector, automative_hexapod:JST-XH-SMD-3-2.54mm, B.Cu at (266.4, 131.3)
- added J13: Connector, automative_hexapod:JST-XH-SMD-3-2.54mm, B.Cu at (266.4, 143.3)
- added J14: Connector, automative_hexapod:JST-XH-SMD-3-2.54mm, B.Cu at (252.4, 83.5)
- added J15: Connector, automative_hexapod:JST-XH-SMD-3-2.54mm, B.Cu at (252.4, 95.5)
- added J16: Connector, automative_hexapod:JST-XH-SMD-3-2.54mm, B.Cu at (252.4, 107.4)
- added J17: Connector, automative_hexapod:JST-XH-SMD-3-2.54mm, B.Cu at (252.4, 119.4)
- added J18: Connector, automative_hexapod:JST-XH-SMD-3-2.54mm, B.Cu at (252.4, 131.3)
- added J19: Connector, automative_hexapod:JST-XH-SMD-3-2.54mm, B.Cu at (252.4, 143.3)
- added J20: Connector, automative_hexapod:JST-XH-SMD-3-2.54mm, B.Cu at (238.3, 83.5)
- added J21: Connector, automative_hexapod:JST-XH-SMD-3-2.54mm, B.Cu at (238.3, 95.5)
- added J22: Connector, automative_hexapod:JST-XH-SMD-3-2.54mm, B.Cu at (238.3, 107.4)
- added J23: Connector, automative_hexapod:JST-XH-SMD-3-2.54mm, B.Cu at (238.3, 119.4)
- added J24: Connector, automative_hexapod:JST-XH-SMD-3-2.54mm, B.Cu at (238.3, 131.3)
- added J25: Connector, automative_hexapod:JST-XH-SMD-3-2.54mm, B.Cu at (238.3, 143.3)
- added J26: Connector, automative_hexapod:JST-XH-SMD-3-2.54mm, B.Cu at (224.3, 83.5)
- added J27: Connector, automative_hexapod:JST-XH-SMD-3-2.54mm, B.Cu at (224.3, 95.5)
- added J28: Connector, automative_hexapod:JST-XH-SMD-3-2.54mm, B.Cu at (224.3, 107.4)
- added J7: Connector, automative_hexapod:JST-XH-SMD-3-2.54mm, B.Cu at (266.4, 83.5)
- added J8: Connector, automative_hexapod:JST-XH-SMD-3-2.54mm, B.Cu at (266.4, 95.5)
- added J9: Connector, automative_hexapod:JST-XH-SMD-3-2.54mm, B.Cu at (266.4, 107.4)
- added R15: 10kOhm, automative_hexapod:Res_0603, B.Cu at (243.7, 38.4)
- added R16: 10kOhm, automative_hexapod:Res_0603, B.Cu at (243.7, 40.5)
- added R20: 10kOhm, automative_hexapod:Res_0603, B.Cu at (240.1, 38.4)
- added R21: 10kOhm, automative_hexapod:Res_0603, B.Cu at (240.1, 40.5)
- added R22: 220Ohm, automative_hexapod:R_Array_Convex_4x0603, B.Cu at (204.3, 66.5)
- added R23: 220Ohm, automative_hexapod:R_Array_Convex_4x0603, B.Cu at (215.9, 66.5)
- added R24: 220Ohm, automative_hexapod:R_Array_Convex_4x0603, B.Cu at (212.0, 66.5)
- added R25: 220Ohm, automative_hexapod:R_Array_Convex_4x0603, B.Cu at (208.2, 66.5)
- added R26: 4.7Ohm, automative_hexapod:Res_0603, B.Cu at (227.4, 51.2)
- added R27: 10kOhm, automative_hexapod:Res_0603, B.Cu at (227.4, 53.3)
- added SW1: MTS-103, automative_hexapod:MTS-103_JCV, B.Cu at (186.1, 125.7)
- added TP1: ~, automative_hexapod:SolderBridgeOpen, B.Cu at (233.1, 38.9)
- added TP2: ~, automative_hexapod:SolderBridgeOpen, B.Cu at (233.1, 42.1)
- added TP3: ~, automative_hexapod:SolderBridgeOpen, B.Cu at (233.1, 45.3)
- added TP4: ~, automative_hexapod:SolderBridgeOpen, B.Cu at (229.9, 38.9)
- added TP5: ~, automative_hexapod:SolderBridgeOpen, B.Cu at (229.9, 42.1)
- added TP6: ~, automative_hexapod:SolderBridgeOpen, B.Cu at (229.9, 45.3)
- added U3: PCA9685PW, automative_hexapod:TSSOP-28_4.4x9.7mm_P0.65mm, B.Cu at (95.6, 141.1)
- C1: value 10uF/16V -> 220uF; footprint automative_hexapod:Ceramic_Cap_0805 -> Capacitor_SMD:CP_Elec_10x10.5; moved to B.Cu
- C10, C8: value 100nF/50V -> 22uF; footprint automative_hexapod:Ceramic_Cap_0805 -> automative_hexapod:Ceramic_Cap_1206; moved to B.Cu
- C11, C30: value 100nF/50V -> 100nF; moved to B.Cu
- C12: value 10uF/16V -> 100nF; moved to B.Cu
- C13, C14, C19, C20, C21, C22, C27, C28: value 10uF/16V -> 10uF; footprint automative_hexapod:Ceramic_Cap_0805 -> automative_hexapod:Ceramic_Cap_0603; moved to B.Cu
- C15, C16, C17, C18, C23, C24, C25, C26: value 100nF/50V -> 100nF; footprint automative_hexapod:Ceramic_Cap_0805 -> automative_hexapod:Ceramic_Cap_0603; moved to B.Cu
- C2: value 100nF/50V -> 220uF; footprint automative_hexapod:Ceramic_Cap_0805 -> Capacitor_SMD:CP_Elec_10x10.5
- C29: value 330uF/50V -> 10uF; footprint Capacitor_SMD:CP_Elec_10x10.5 -> automative_hexapod:Ceramic_Cap_0805; moved to B.Cu
- C3: value 10uF/16V -> 1uF; footprint automative_hexapod:Ceramic_Cap_0805 -> automative_hexapod:Ceramic_Cap_1206; moved to B.Cu
- C31, C37: value 10uF/16V -> 10uF; moved to B.Cu
- C38: value 220uF/50V -> 10uF; footprint Capacitor_SMD:CP_Elec_10x10.5 -> automative_hexapod:Ceramic_Cap_0805; moved to B.Cu
- C39: value 100nF/50V -> 10uF; moved to B.Cu
- C4: value 100nF/50V -> 1uF; footprint automative_hexapod:Ceramic_Cap_0805 -> automative_hexapod:Ceramic_Cap_1206; moved to B.Cu
- C45, C46: value 1uF/16V -> 100nF; moved to B.Cu
- C5: value 10uF/16V -> 330uF; footprint automative_hexapod:Ceramic_Cap_0805 -> Capacitor_SMD:CP_Elec_10x10.5; moved to B.Cu
- C6: value 100nF/50V -> 330uF; footprint automative_hexapod:Ceramic_Cap_0805 -> Capacitor_SMD:CP_Elec_10x10.5
- C7, C9: value 10uF/16V -> 22uF; footprint automative_hexapod:Ceramic_Cap_0805 -> automative_hexapod:Ceramic_Cap_1206; moved to B.Cu
- D1: value LED_0805 -> PIN; moved to B.Cu
- D2: value MBR20100CT -> 5V; footprint automative_hexapod:TO-220-3 -> automative_hexapod:LED_0805
- J1: value MPU6050 -> Pin Connector; footprint automative_hexapod:MPU6050 -> automative_hexapod:Connector-Pin
- J2, J3: value Conn_01x04_Pin -> Connector; footprint automative_hexapod:PinHeader_1x04_P2.54mm_Vertical -> automative_hexapod:TerminalBlock_Phoenix_MKDS-1,5-4-5.08_1x04_P5.08mm_Horizontal
- J4: value Conn_01x04_Pin -> MPU6050; footprint automative_hexapod:PinHeader_1x04_P2.54mm_Vertical -> automative_hexapod:MPU6050; moved to F.Cu
- L1, Q1, Q2, Q3, Q4, Q5: moved to B.Cu
- R1, R4: value 10K/1%/1/8W -> 10.5kOhm; moved to B.Cu
- R10, R11, R12, R17, R19, R7, R8, R9: value 10K/1%/1/8W -> 10kOhm; footprint automative_hexapod:Res_0805 -> automative_hexapod:Res_0603; moved to B.Cu
- R13: value 10.5K/1%/1/8W -> 10kOhm; footprint automative_hexapod:Res_0805 -> automative_hexapod:Res_0603; moved to B.Cu
- R14: value 2K/1%/1/8W -> 10kOhm; footprint automative_hexapod:Res_0805 -> automative_hexapod:Res_0603; moved to B.Cu
- R18: value 1K/1%/1/8W -> 10kOhm; footprint automative_hexapod:Res_0805 -> automative_hexapod:Res_0603; moved to B.Cu
- R2: value 10K/1%/1/8W -> 5.6kOhm; moved to B.Cu
- R3, R5: value 10K/1%/1/8W -> 2kOhm; moved to B.Cu
- R6: value 10K/1%/1/8W -> 1K/1%/1/8W; moved to B.Cu
- U1: value ~ -> XL4005E1; footprint automative_hexapod:BeagleBone_AI -> automative_hexapod:TO-263-5; moved to B.Cu
- U2: value XL4005E1 -> ~; footprint automative_hexapod:TO-263-5 -> automative_hexapod:BeagleBone_AI; moved to B.Cu
- moved C14 215.0 mm to (243.7, 14.4), turned to 180 degrees
- moved C20 212.4 mm to (236.6, 14.4)
- moved C18 212.0 mm to (240.1, 18.7)
- moved R5 209.8 mm to (263.2, 44.0), turned to 180 degrees
- moved C16 209.3 mm to (243.7, 23.0), turned to 180 degrees
- moved C13 207.6 mm to (243.7, 12.3), turned to 180 degrees
- moved C19 205.0 mm to (236.6, 12.3)
- moved C17 205.0 mm to (240.1, 16.5)
- moved R8 204.3 mm to (229.4, 14.4), turned to 180 degrees
- moved C15 202.6 mm to (243.7, 20.8), turned to 180 degrees
- moved R1 202.4 mm to (263.2, 33.7), turned to 180 degrees
- moved R7 197.0 mm to (229.4, 12.3), turned to 180 degrees
- moved Q4 197.0 mm to (219.9, 8.76), turned to 180 degrees
- moved Q1 195.9 mm to (243.2, 8.76), turned to 180 degrees
- moved R2 195.4 mm to (263.2, 36.3), turned to 180 degrees
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Connections:
- C1 pad 1: GND -> VCC
- C1 pad 2: +5V -> GND
- C12 pad 2: +5V -> +3.3V
- C2 pad 1: GND -> VCC
- C2 pad 2: +5V -> GND
- C29 pad 1: +5V -> GND
- C29 pad 2: GND -> +5V
- C3 pad 2: +3.3V -> VCC
- C37 pad 2: +3.3V -> +5V
- C38 pad 1: VCC -> GND
- C38 pad 2: GND -> +5V
- C39 pad 2: +3.3V -> +5V
- C4 pad 2: +3.3V -> +5V
- C45 pad 2: VCC -> +5V
- C5 pad 1: GND -> +5V
- C5 pad 2: +3.3V -> GND
- C6 pad 1: GND -> +5V
- C6 pad 2: +3.3V -> GND
- C8 pad 2: +5V -> +3.3V
- C9 pad 2: +3.3V -> +5V
- D1 pad 1: GND -> Net-(D1-K)
- D1 pad 2: Net-(D1-A) -> VCC
- D2 pad 1: GND -> Net-(D2-K)
- D2 pad 2: Net-(U2-SW) -> +5V
- J1 pad 1: +5V -> unconnected-(J1-Pin_1-Pad1)
- J1 pad 2: GND -> unconnected-(J1-Pin_2-Pad2)
- J2 pad 1: +5V -> unconnected-(J2-Pin_1-Pad1)
- J2 pad 2: GND -> unconnected-(J2-Pin_2-Pad2)
- J2 pad 3: PCA9685_I2C_SCL -> unconnected-(J2-Pin_3-Pad3)
- J2 pad 4: PCA9685_I2C_SDA -> unconnected-(J2-Pin_4-Pad4)
- J3 pad 1: +5V -> unconnected-(J3-Pin_1-Pad1)
- J3 pad 2: GND -> unconnected-(J3-Pin_2-Pad2)
- J3 pad 3: PCA9685_I2C_SDA -> unconnected-(J3-Pin_3-Pad3)
- J3 pad 4: PCA9685_I2C_SCL -> unconnected-(J3-Pin_4-Pad4)
- J4 pad 3: HCSR04_ECHO -> MPU6050_I2C_SCL
- J4 pad 4: HCSR04_TRIG -> MPU6050_I2C_SDA
- L1 pad 1: Net-(U2-SW) -> Net-(U1-SW)
- Q1 pad 2: BBAI_I2C_SCL -> BBAI_TRIG
- Q1 pad 3: MPU6050_I2C_SCL -> HCSR04_TRIG
- Q2 pad 2: BBAI_I2C_SDA -> BBAI_ECHO
- Q2 pad 3: MPU6050_I2C_SDA -> HCSR04_ECHO
- Q5 pad 1: +3.3V -> Net-(Q5-G)
- Q5 pad 2: BBAI_TRIG -> GND
- Q5 pad 3: HCSR04_TRIG -> unconnected-(Q5-D-Pad3)
- R1 pad 1: BBAI_I2C_SCL -> GND
- R1 pad 2: +3.3V -> Net-(D1-K)
- R10 pad 1: BBAI_ECHO -> HCSR04_ECHO
- R10 pad 2: +3.3V -> +5V
- R11 pad 1: HCSR04_TRIG -> BBAI_I2C_SDA
- R11 pad 2: +5V -> +3.3V
- R12 pad 1: HCSR04_ECHO -> BBAI_I2C_SCL
- R12 pad 2: +5V -> +3.3V
- R13 pad 1: Net-(U2-FB) -> PCA9685_I2C_SDA
- R14 pad 1: GND -> PCA9685_I2C_SCL
- R14 pad 2: Net-(U2-FB) -> +5V
- R17 pad 1: BBAI_PWM1A -> GND
- R17 pad 2: +3.3V -> /Servo Drivers/A2_0
- R18 pad 1: Net-(U1-GPIO0_26) -> GND
- R18 pad 2: Net-(D1-A) -> /Servo Drivers/A3_0
- R19 pad 1: FAN_PWM1A -> GND
- R19 pad 2: +5V -> /Servo Drivers/A4_0
- R2 pad 1: MPU6050_I2C_SCL -> GND
- R2 pad 2: +5V -> Net-(D2-K)
- R3 pad 1: BBAI_I2C_SDA -> GND
- R3 pad 2: +3.3V -> Net-(D3-K)
- R4 pad 1: MPU6050_I2C_SDA -> Net-(U1-FB)
- R5 pad 1: BBAI_I2C_SDA -> GND
- R5 pad 2: +3.3V -> Net-(U1-FB)
- R6 pad 1: BBAI_I2C_SCL -> Net-(U2-GPIO0_26)
- R6 pad 2: +3.3V -> Net-(D5-A)
- R7 pad 1: PCA9685_I2C_SDA -> BBAI_TRIG
- R7 pad 2: +5V -> +3.3V
- R8 pad 1: PCA9685_I2C_SCL -> BBAI_ECHO
- R8 pad 2: +5V -> +3.3V
- R9 pad 1: BBAI_TRIG -> HCSR04_TRIG
- R9 pad 2: +3.3V -> +5V
Routing:
- net GND: track 625.0 -> 0.00 mm, vias 19 -> 0
- net +3.3V: track 369.4 -> 0.00 mm, vias 14 -> 0
- net +5V: track 355.1 -> 0.00 mm, vias 9 -> 0
- net BBAI_I2C_SDA: track 100.7 -> 0.00 mm
- net BBAI_PWM1A: track 86.7 -> 0.00 mm
- net BBAI_I2C_SCL: track 69.8 -> 0.00 mm
- net Net-(U2-SW): track 32.3 -> 0.00 mm
- net PCA9685_I2C_SCL: track 28.3 -> 0.00 mm
- net PCA9685_I2C_SDA: track 22.4 -> 0.00 mm
- net VCC: track 22.3 -> 0.00 mm, vias 1 -> 0
- net BBAI_ECHO: track 19.4 -> 0.00 mm
- net HCSR04_ECHO: track 18.4 -> 0.00 mm
- net BBAI_TRIG: track 14.7 -> 0.00 mm
- net Net-(U2-FB): track 12.0 -> 0.00 mm
- net MPU6050_I2C_SDA: track 10.4 -> 0.00 mm
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- removed copper zone on F.Cu, net +5V
- removed copper zone on F.Cu, net VCC
Other:
- board size 110.1 x 111.8 mm -> 100 x 100 mm
