File: hardware/Source/Ver_1.1.0/Automative_Hexapod.kicad_pcb (KiCad board)
At the start: 2 copper layers, 110.1 x 111.8 mm, 70 parts, among them J1 MPU6050, J2 Conn_01x04_Pin, J3 Conn_01x04_Pin, J4 Conn_01x04_Pin, J5 Conn_01x03_Pin, Q1 LN2302LT1G, Q2 LN2302LT1G, Q3 LN2302LT1G, Q4 LN2302LT1G, Q5 LN2302LT1G, Q6 LN2302LT1G, Q9 LN2302LT1G, U2 XL4005E1

Commit message: update pcb v1.1.0
Parts:
- removed Q6, Q9: LN2302LT1G, automative_hexapod:SOT23
- added C32: 100nF, automative_hexapod:Ceramic_Cap_0805, B.Cu at (24.5, 30.1)
- added C33: 10uF, automative_hexapod:Ceramic_Cap_0805, F.Cu at (94.4, 136.0)
- added C34: 100nF, automative_hexapod:Ceramic_Cap_0805, F.Cu at (94.4, 138.7)
- added C35: 10uF, automative_hexapod:Ceramic_Cap_0805, B.Cu at (91.9, 73.8)
- added C36: 100nF, automative_hexapod:Ceramic_Cap_0805, B.Cu at (91.9, 76.5)
- added C40: 10uF, automative_hexapod:Ceramic_Cap_0805, F.Cu at (137.0, 88.2)
- added C41: 10uF, automative_hexapod:Ceramic_Cap_0805, F.Cu at (137.0, 80.0)
- added C42: 10uF, automative_hexapod:Ceramic_Cap_0805, F.Cu at (137.0, 90.9)
- added C43: 10uF, automative_hexapod:Ceramic_Cap_0805, B.Cu at (135.5, 118.5)
- added C44: 100nF, automative_hexapod:Ceramic_Cap_0805, F.Cu at (141.0, 77.3)
- added C47: 100nF, automative_hexapod:Ceramic_Cap_0805, F.Cu at (141.0, 82.8)
- added C48: 100nF, automative_hexapod:Ceramic_Cap_0805, B.Cu at (135.4, 121.0)
- added C49: 10uF, automative_hexapod:Ceramic_Cap_0805, B.Cu at (120.0, 135.0)
- added C50: 10uF, automative_hexapod:Ceramic_Cap_0805, B.Cu at (113.7, 147.8)
- added C51: 10uF, automative_hexapod:Ceramic_Cap_0805, F.Cu at (135.2, 123.9)
- added C52: 10uF, automative_hexapod:Ceramic_Cap_0805, F.Cu at (136.1, 136.3)
- added C53: 100nF, automative_hexapod:Ceramic_Cap_0805, B.Cu at (120.0, 137.0)
- added C54: 100nF, automative_hexapod:Ceramic_Cap_0805, B.Cu at (113.7, 150.6)
- added C55: 100nF, automative_hexapod:Ceramic_Cap_0805, F.Cu at (135.2, 126.0)
- added C56: 100nF, automative_hexapod:Ceramic_Cap_0805, F.Cu at (136.1, 138.6)
- added C57: 10uF, automative_hexapod:Ceramic_Cap_0805, F.Cu at (108.4, 150.9)
- added C58: 10uF, automative_hexapod:Ceramic_Cap_0805, B.Cu at (36.6, 62.6)
- added C59: 10uF, automative_hexapod:Ceramic_Cap_0805, B.Cu at (36.6, 65.4)
- added C60: 10uF, automative_hexapod:Ceramic_Cap_0805, B.Cu at (36.6, 68.1)
- added C61: 10uF, automative_hexapod:Ceramic_Cap_0805, B.Cu at (36.6, 70.8)
- added C62: 100nF, automative_hexapod:Ceramic_Cap_0805, F.Cu at (108.7, 149.0)
- added C63: 100nF, automative_hexapod:Ceramic_Cap_0805, B.Cu at (36.6, 76.2)
- added C64: 100nF, automative_hexapod:Ceramic_Cap_0805, B.Cu at (36.6, 79.0)
- added C65: 100nF, automative_hexapod:Ceramic_Cap_0805, B.Cu at (32.6, 62.6)
- added C66: 100nF, automative_hexapod:Ceramic_Cap_0805, B.Cu at (32.6, 65.4)
- added C67: 10uF, automative_hexapod:Ceramic_Cap_0805, B.Cu at (32.6, 68.1)
- added C68: 10uF, automative_hexapod:Ceramic_Cap_0805, B.Cu at (32.6, 70.8)
- added C69: 10uF, automative_hexapod:Ceramic_Cap_0805, B.Cu at (32.6, 73.5)
- added C70: 10uF, automative_hexapod:Ceramic_Cap_0805, B.Cu at (32.6, 76.2)
- added C71: 100nF, automative_hexapod:Ceramic_Cap_0805, B.Cu at (32.6, 79.0)
- added C72: 100nF, automative_hexapod:Ceramic_Cap_0805, B.Cu at (28.5, 62.6)
- added C73: 100nF, automative_hexapod:Ceramic_Cap_0805, B.Cu at (28.5, 65.4)
- added C74: 100nF, automative_hexapod:Ceramic_Cap_0805, B.Cu at (28.5, 68.1)
- added C75: 47uF, automative_hexapod:Ceramic_Cap_1206, F.Cu at (30.1, 115.2)
- added C76: 47uF, automative_hexapod:Ceramic_Cap_1206, F.Cu at (32.4, 115.2)
- added D3: 5V, automative_hexapod:LED_0805, F.Cu at (160.2, 96.8)
- added D4: 3.3V, automative_hexapod:LED_0805, F.Cu at (160.2, 99.8)
- added D5: SS54, automative_hexapod:D_SMA, F.Cu at (35.1, 116.4)
- added D6: LED_0805, automative_hexapod:LED_0805, F.Cu at (131.2, 59.4)
- added F1: Fuse, automative_hexapod:FUSE_SMD_1808, F.Cu at (69.0, 120.9)
- added J10: Connector, automative_hexapod:JST-XH-SMD-3-2.54mm, B.Cu at (125.1, 110.8)
- added J11: Connector, automative_hexapod:JST-XH-SMD-3-2.54mm, B.Cu at (125.1, 124.0)
- added J12: Connector, automative_hexapod:JST-XH-SMD-3-2.54mm, B.Cu at (125.1, 137.2)
- added J13: Connector, automative_hexapod:JST-XH-SMD-3-2.54mm, B.Cu at (111.2, 137.0)
- added J14: Connector, automative_hexapod:JST-XH-SMD-3-2.54mm, F.Cu at (125.1, 124.0)
- added J15: Connector, automative_hexapod:JST-XH-SMD-3-2.54mm, F.Cu at (125.1, 137.2)
- added J16: Connector, automative_hexapod:JST-XH-SMD-3-2.54mm, F.Cu at (111.2, 137.0)
- added J17: Connector, automative_hexapod:JST-XH-SMD-3-2.54mm, B.Cu at (63.0, 104.1)
- added J18: Connector, automative_hexapod:JST-XH-SMD-3-2.54mm, B.Cu at (63.0, 91.0)
- added J19: Connector, automative_hexapod:JST-XH-SMD-3-2.54mm, B.Cu at (63.0, 77.8)
- added J20: Connector, automative_hexapod:JST-XH-SMD-3-2.54mm, B.Cu at (63.0, 64.7)
- added J21: Connector, automative_hexapod:JST-XH-SMD-3-2.54mm, B.Cu at (63.0, 51.5)
- added J22: Connector, automative_hexapod:JST-XH-SMD-3-2.54mm, B.Cu at (80.2, 52.8)
- added J23: Connector, automative_hexapod:JST-XH-SMD-3-2.54mm, F.Cu at (80.2, 52.8)
- added J24: Connector, automative_hexapod:JST-XH-SMD-3-2.54mm, F.Cu at (93.6, 52.9)
- added J6: Connector, automative_hexapod:JST-XH-SMD-4-2.54mm, B.Cu at (115.4, 53.0)
- added J7: Connector, automative_hexapod:JST-XH-SMD-3-2.54mm, B.Cu at (125.1, 71.4)
- added J8: Connector, automative_hexapod:JST-XH-SMD-3-2.54mm, B.Cu at (125.1, 84.6)
- added J9: Connector, automative_hexapod:JST-XH-SMD-3-2.54mm, B.Cu at (125.1, 97.7)
- added R15: 10kOhm, automative_hexapod:Res_0603, B.Cu at (150.0, 61.8)
- added R16: 10kOhm, automative_hexapod:Res_0603, B.Cu at (165.9, 13.0)
- added R20: 10kOhm, automative_hexapod:Res_0603, B.Cu at (165.9, 17.3)
- added R21: 10kOhm, automative_hexapod:Res_0603, B.Cu at (37.0, 20.4)
- added R22: 10kOhm, automative_hexapod:Res_0603, B.Cu at (165.9, 19.5)
- added R23: 10kOhm, automative_hexapod:Res_0603, B.Cu at (37.0, 22.6)
- added R24: 10kOhm, automative_hexapod:Res_0603, B.Cu at (165.9, 21.6)
- added R25: 10kOhm, automative_hexapod:Res_0603, B.Cu at (37.0, 24.8)
- added R26: 10kOhm, automative_hexapod:Res_0603, B.Cu at (162.3, 13.0)
- added R27: 10kOhm, automative_hexapod:Res_0603, B.Cu at (37.0, 26.9)
- added R28: 10kOhm, automative_hexapod:Res_0603, B.Cu at (162.3, 15.1)
- added R29: 10kOhm, automative_hexapod:Res_0603, B.Cu at (37.0, 29.1)
- added R30: 220Ohm, automative_hexapod:R_Array_Convex_4x0603, B.Cu at (144.8, 24.4)
- added R31: 220Ohm, automative_hexapod:R_Array_Convex_4x0603, B.Cu at (148.7, 29.3)
- added R32: 220Ohm, automative_hexapod:R_Array_Convex_4x0603, B.Cu at (33.3, 17.3)
- added R33: 220Ohm, automative_hexapod:R_Array_Convex_4x0603, B.Cu at (29.5, 17.3)
- added R34: 220Ohm, automative_hexapod:R_Array_Convex_4x0603, B.Cu at (144.9, 29.3)
- added R35: 220Ohm, automative_hexapod:R_Array_Convex_4x0603, B.Cu at (25.6, 17.3)
- added R36: 4.7Ohm, automative_hexapod:Res_0603, B.Cu at (95.8, 71.3)
- added R37: 10kOhm, automative_hexapod:Res_0603, B.Cu at (95.8, 73.4)
- added R38: 10kOhm, automative_hexapod:Res_0603, B.Cu at (91.9, 71.5)
- added R39: 30kOhm, automative_hexapod:Res_0603, F.Cu at (40.7, 111.1)
- added R40: 2.49kOhm, automative_hexapod:Res_0603, F.Cu at (40.7, 106.9)
- added R41: 49.9kOhm, automative_hexapod:Res_0603, F.Cu at (40.6, 108.3)
- added R42: 10kOhm, automative_hexapod:Res_0603, F.Cu at (40.7, 109.7)
- added SW1: MTS-102-C3, automative_hexapod:MTS-102-C3, F.Cu at (70.0, 137.9)
- added TP1: ~, automative_hexapod:SolderBridgeOpen, B.Cu at (155.3, 13.5)
- added TP10: ~, automative_hexapod:SolderBridgeOpen, B.Cu at (18.4, 21.1)
- added TP11: ~, automative_hexapod:SolderBridgeOpen, B.Cu at (152.1, 20.0)
- added TP12: ~, automative_hexapod:SolderBridgeOpen, B.Cu at (18.4, 24.4)
- added TP2: ~, automative_hexapod:SolderBridgeOpen, B.Cu at (24.9, 21.1)
- added TP3: ~, automative_hexapod:SolderBridgeOpen, B.Cu at (155.3, 16.7)
- added TP4: ~, automative_hexapod:SolderBridgeOpen, B.Cu at (24.9, 24.4)
- added TP5: ~, automative_hexapod:SolderBridgeOpen, B.Cu at (155.3, 20.0)
- added TP6: ~, automative_hexapod:SolderBridgeOpen, B.Cu at (21.7, 21.1)
- added TP7: ~, automative_hexapod:SolderBridgeOpen, B.Cu at (152.1, 13.5)
- added TP8: ~, automative_hexapod:SolderBridgeOpen, B.Cu at (21.7, 24.4)
- added TP9: ~, automative_hexapod:SolderBridgeOpen, B.Cu at (152.1, 16.7)
- added U3: PCA9685PW, automative_hexapod:TSSOP-28_4.4x9.7mm_P0.65mm, B.Cu at (156.1, 32.7)
- added U4: PCA9685PW, automative_hexapod:TSSOP-28_4.4x9.7mm_P0.65mm, B.Cu at (30.9, 25.2)
- C1: value 10uF/16V -> 100uF; footprint automative_hexapod:Ceramic_Cap_0805 -> automative_hexapod:CP_Elec_6.3x5.4
- C10, C8: value 100nF/50V -> 22uF; footprint automative_hexapod:Ceramic_Cap_0805 -> automative_hexapod:Ceramic_Cap_1206
- C11, C2: value 100nF/50V -> 100nF; footprint automative_hexapod:Ceramic_Cap_0805 -> automative_hexapod:Ceramic_Cap_1206
- C12: value 10uF/16V -> 100nF; footprint automative_hexapod:Ceramic_Cap_0805 -> automative_hexapod:Ceramic_Cap_1206
- C13, C14, C19, C20, C21, C22, C27, C28: value 10uF/16V -> 10uF; footprint automative_hexapod:Ceramic_Cap_0805 -> automative_hexapod:Ceramic_Cap_0603; moved to B.Cu
- C15, C16, C17, C18, C23, C24, C25, C26: value 100nF/50V -> 100nF; footprint automative_hexapod:Ceramic_Cap_0805 -> automative_hexapod:Ceramic_Cap_0603; moved to B.Cu
- C29: value 330uF/50V -> 10uF; footprint Capacitor_SMD:CP_Elec_10x10.5 -> automative_hexapod:Ceramic_Cap_0805; moved to B.Cu
- C3: value 10uF/16V -> 4.7nF; footprint automative_hexapod:Ceramic_Cap_0805 -> automative_hexapod:Ceramic_Cap_0603
- C30: value 100nF/50V -> 10uF; moved to B.Cu
- C31: value 10uF/16V -> 100nF; moved to B.Cu
- C37: value 10uF/16V -> 10uF; moved to B.Cu
- C38: value 220uF/50V -> 100nF; footprint Capacitor_SMD:CP_Elec_10x10.5 -> automative_hexapod:Ceramic_Cap_0805; moved to B.Cu
- C39: value 100nF/50V -> 10uF
- C4: value 100nF/50V -> 39pF; footprint automative_hexapod:Ceramic_Cap_0805 -> automative_hexapod:Ceramic_Cap_0603
- C45, C46: value 1uF/16V -> 100nF
- C5: value 10uF/16V -> 10nF; footprint automative_hexapod:Ceramic_Cap_0805 -> automative_hexapod:Ceramic_Cap_0603
- C6: value 100nF/50V -> 100nF; footprint automative_hexapod:Ceramic_Cap_0805 -> automative_hexapod:Ceramic_Cap_0603
- C7, C9: value 10uF/16V -> 22uF; footprint automative_hexapod:Ceramic_Cap_0805 -> automative_hexapod:Ceramic_Cap_1206
- D1: value LED_0805 -> PIN
- D2: value MBR20100CT -> PIN; footprint automative_hexapod:TO-220-3 -> automative_hexapod:LED_0805; moved to F.Cu
- J1: value MPU6050 -> Pin Connector; footprint automative_hexapod:MPU6050 -> automative_hexapod:Connector-Pin; moved to F.Cu
- J2, J3: value Conn_01x04_Pin -> Connector; footprint automative_hexapod:PinHeader_1x04_P2.54mm_Vertical -> automative_hexapod:TerminalBlock_Phoenix_MKDS-1,5-4-5.08_1x04_P5.08mm_Horizontal; moved to F.Cu
- J4: value Conn_01x04_Pin -> MPU6050; footprint automative_hexapod:PinHeader_1x04_P2.54mm_Vertical -> automative_hexapod:MPU6050
- J5: value Conn_01x03_Pin -> Connector; footprint automative_hexapod:PinHeader_1x03_P2.54mm_Vertical -> automative_hexapod:JST-XH-SMD-2-2.54mm
- L1: value 27uH 5.7A -> 10uH 4A; footprint automative_hexapod:IND_CDRH127_LDNP-470MC_SUM -> automative_hexapod:Inductor_0630
- Q1, Q2, Q3, Q4, Q5: moved to B.Cu
- R1, R2: value 10K/1%/1/8W -> 10.5kOhm
- R10, R11, R12, R17, R19, R8, R9: value 10K/1%/1/8W -> 10kOhm; footprint automative_hexapod:Res_0805 -> automative_hexapod:Res_0603; moved to B.Cu
- R13: value 10.5K/1%/1/8W -> 10kOhm; footprint automative_hexapod:Res_0805 -> automative_hexapod:Res_0603; moved to B.Cu
- R14: value 2K/1%/1/8W -> 10kOhm; footprint automative_hexapod:Res_0805 -> automative_hexapod:Res_0603; moved to B.Cu
- R18: value 1K/1%/1/8W -> 10kOhm; footprint automative_hexapod:Res_0805 -> automative_hexapod:Res_0603; moved to B.Cu
- R3: value 10K/1%/1/8W -> 5.6kOhm
- R4: value 10K/1%/1/8W -> 2kOhm
- R5: value 10K/1%/1/8W -> 100kOhm; footprint automative_hexapod:Res_0805 -> automative_hexapod:Res_0603
- R6: value 10K/1%/1/8W -> 20kOhm; footprint automative_hexapod:Res_0805 -> automative_hexapod:Res_0603
- R7: value 10K/1%/1/8W -> 1K/1%/1/8W
- U1: value ~ -> TPS54331DR; footprint automative_hexapod:BeagleBone_AI -> automative_hexapod:SOIC-8
- U2: value XL4005E1 -> ~; footprint automative_hexapod:TO-263-5 -> automative_hexapod:BeagleBone_AI
- moved C30 133.9 mm to (24.5, 27.3), turned to 180 degrees
- moved R19 132.2 mm to (37.0, 18.3), turned to 180 degrees
- moved C14 131.0 mm to (171.5, 57.4), turned to 180 degrees
- moved R17 128.6 mm to (37.0, 16.1), turned to 180 degrees
- moved C20 128.5 mm to (164.4, 57.4)
- moved C18 127.9 mm to (168.0, 61.7)
- moved C16 125.3 mm to (171.5, 66.0), turned to 180 degrees
- moved C13 123.7 mm to (171.5, 55.3), turned to 180 degrees
- moved R8 121.5 mm to (157.2, 55.3), turned to 180 degrees
- moved C17 121.2 mm to (168.0, 59.6)
- moved C19 121.0 mm to (164.4, 55.3)
- moved C15 119.0 mm to (171.5, 63.9), turned to 180 degrees
- moved Q4 113.4 mm to (147.7, 51.8), turned to 180 degrees
- moved Q1 112.7 mm to (171.0, 51.8), turned to 180 degrees
- moved L1 109.0 mm to (33.7, 109.2), turned to 180 degrees
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Connections:
- C1 pad 1: GND -> VCC
- C1 pad 2: +5V -> GND
- C11 pad 1: GND -> +5V
- C11 pad 2: +5V -> GND
- C12 pad 1: GND -> +3.3V
- C12 pad 2: +5V -> GND
- C2 pad 1: GND -> VCC
- C2 pad 2: +5V -> GND
- C29 pad 1: +5V -> GND
- C29 pad 2: GND -> +5V
- C3 pad 1: GND -> Net-(C3-Pad1)
- C3 pad 2: +3.3V -> Net-(U1-COMP)
- C37 pad 2: +3.3V -> +5V
- C38 pad 1: VCC -> GND
- C38 pad 2: GND -> +5V
- C39 pad 2: +3.3V -> Vdrive
- C4 pad 2: +3.3V -> Net-(U1-COMP)
- C45 pad 2: VCC -> Vdrive
- C46 pad 2: +5V -> Vdrive
- C5 pad 2: +3.3V -> Net-(U1-SS)
- C6 pad 1: GND -> Net-(U1-BOOT)
- C6 pad 2: +3.3V -> Net-(D5-K)
- C8 pad 2: +5V -> +3.3V
- C9 pad 2: +3.3V -> +5V
- D1 pad 1: GND -> Net-(D1-K)
- D1 pad 2: Net-(D1-A) -> +BATT
- D2 pad 1: GND -> Net-(D2-K)
- D2 pad 2: Net-(U2-SW) -> VCC
- J1 pad 1: +5V -> Net-(J1-Pin_1)
- J2 pad 1: +5V -> +BATT
- J2 pad 2: GND -> +BATT
- J2 pad 3: PCA9685_I2C_SCL -> GND
- J2 pad 4: PCA9685_I2C_SDA -> GND
- J3 pad 1: +5V -> Vdrive
- J3 pad 2: GND -> Vdrive
- J3 pad 3: PCA9685_I2C_SDA -> GND
- J3 pad 4: PCA9685_I2C_SCL -> GND
- J4 pad 3: HCSR04_ECHO -> MPU6050_I2C_SCL
- J4 pad 4: HCSR04_TRIG -> MPU6050_I2C_SDA
- J5 pad 1: +5V -> Net-(J5-Pin_1)
- J5 pad 2: GND -> Net-(J5-Pin_2)
- L1 pad 1: Net-(U2-SW) -> Net-(D5-K)
- Q1 pad 2: BBAI_I2C_SCL -> BBAI_TRIG
- Q1 pad 3: MPU6050_I2C_SCL -> HCSR04_TRIG
- Q2 pad 2: BBAI_I2C_SDA -> BBAI_ECHO
- Q2 pad 3: MPU6050_I2C_SDA -> HCSR04_ECHO
- Q5 pad 1: +3.3V -> Net-(Q5-G)
- Q5 pad 2: BBAI_TRIG -> GND
- Q5 pad 3: HCSR04_TRIG -> Net-(J5-Pin_2)
- R1 pad 1: BBAI_I2C_SCL -> GND
- R1 pad 2: +3.3V -> Net-(D1-K)
- R10 pad 1: BBAI_ECHO -> HCSR04_TRIG
- R10 pad 2: +3.3V -> +5V
- R11 pad 1: HCSR04_TRIG -> HCSR04_ECHO
- R12 pad 1: HCSR04_ECHO -> BBAI_I2C_SDA
- R12 pad 2: +5V -> +3.3V
- R13 pad 1: Net-(U2-FB) -> BBAI_I2C_SCL
- R13 pad 2: +5V -> +3.3V
- R14 pad 1: GND -> PCA9685_I2C_SDA
- R14 pad 2: Net-(U2-FB) -> +5V
- R17 pad 1: BBAI_PWM1A -> GND
- R17 pad 2: +3.3V -> /Servo Drivers/A1_0
- R18 pad 1: Net-(U1-GPIO0_26) -> GND
- R18 pad 2: Net-(D1-A) -> /Servo Drivers/A0_1
- R19 pad 1: FAN_PWM1A -> GND
- R19 pad 2: +5V -> /Servo Drivers/A1_1
- R2 pad 1: MPU6050_I2C_SCL -> GND
- R2 pad 2: +5V -> Net-(D2-K)
- R3 pad 1: BBAI_I2C_SDA -> GND
- R3 pad 2: +3.3V -> Net-(D3-K)
- R4 pad 1: MPU6050_I2C_SDA -> GND
- R4 pad 2: +5V -> Net-(D4-K)
- R5 pad 1: BBAI_I2C_SDA -> Net-(U1-EN)
- R5 pad 2: +3.3V -> VCC
- R6 pad 1: BBAI_I2C_SCL -> GND
- R6 pad 2: +3.3V -> Net-(U1-EN)
- R7 pad 1: PCA9685_I2C_SDA -> Net-(U2-GPIO0_26)
- R7 pad 2: +5V -> Net-(D6-A)
- R8 pad 1: PCA9685_I2C_SCL -> BBAI_TRIG
- R8 pad 2: +5V -> +3.3V
- R9 pad 1: BBAI_TRIG -> BBAI_ECHO
Routing:
- net GND: track 625.0 -> 0.00 mm, vias 19 -> 0
- net +3.3V: track 369.4 -> 0.00 mm, vias 14 -> 0
- net +5V: track 355.1 -> 0.00 mm, vias 9 -> 0
- net BBAI_I2C_SDA: track 100.7 -> 0.00 mm
- net BBAI_PWM1A: track 86.7 -> 0.00 mm
- net BBAI_I2C_SCL: track 69.8 -> 0.00 mm
- net Net-(U2-SW): track 32.3 -> 0.00 mm
- net PCA9685_I2C_SCL: track 28.3 -> 0.00 mm
- net PCA9685_I2C_SDA: track 22.4 -> 0.00 mm
- net VCC: track 22.3 -> 0.00 mm, vias 1 -> 0
- net BBAI_ECHO: track 19.4 -> 0.00 mm
- net HCSR04_ECHO: track 18.4 -> 0.00 mm
- net BBAI_TRIG: track 14.7 -> 0.00 mm
- net Net-(U2-FB): track 12.0 -> 0.00 mm
- net MPU6050_I2C_SDA: track 10.4 -> 0.00 mm
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- removed copper zone on F.Cu, net +5V
- removed copper zone on F.Cu, net VCC
Other:
- board size 110.1 x 111.8 mm -> 78 x 100 mm
- rule pad_to_mask_clearance: 0 -> 0.0508

Commit message: update pcb and schematic
Parts:
- removed the C21 at (164.4, 63.9)
- removed the C22 at (164.4, 66.0)
- removed the C27 at (160.8, 63.9)
- removed the C28 at (160.8, 66.0)
- removed the C29 at (165.0, 27.9)
- removed the C30 at (24.5, 27.3)
- removed the C31 at (165.0, 30.6)
- removed the C32 at (24.5, 30.1)
- removed the Q3 at (152.4, 51.8)
- removed Q4: LN2302LT1G, automative_hexapod:SOT23
- removed the R14 at (150.0, 59.6)
- removed the R15 at (150.0, 61.8)
- C15: renamed from C13; moved to F.Cu
- C16: renamed from C14; moved to F.Cu
- C17: renamed from C15; moved to F.Cu
- C18: renamed from C16; moved to F.Cu
- C19: renamed from C17; moved to F.Cu
- C20: renamed from C18; moved to F.Cu
- C21: renamed from C19; moved to F.Cu
- C22: renamed from C20; moved to F.Cu
- C23, C24: value 100nF -> 10uF; moved to F.Cu
- C25, C26, J13, J21, Q1, Q2, R12, R13, TP1, TP10, TP11, TP12, TP2, TP3, TP4, TP5, TP6, TP7, TP8, TP9, U3, U4: moved to F.Cu
- C44: renamed from C50; moved to F.Cu
- C48: renamed from C54; moved to F.Cu
- C52: renamed from C58; moved to F.Cu
- C53: renamed from C59; moved to F.Cu
- C54: renamed from C60; moved to F.Cu
- C57: renamed from C63; moved to F.Cu
- C58: renamed from C64; moved to F.Cu
- C59: renamed from C65; moved to F.Cu
- C61: renamed from C67; moved to F.Cu
- C63: renamed from C69; moved to F.Cu
- C64: renamed from C70; moved to F.Cu
- C65: renamed from C71; moved to F.Cu
- C67: renamed from C73; moved to F.Cu
- C68: renamed from C74; moved to F.Cu
- J16: moved to B.Cu
- R11: renamed from R7; value 1K/1%/1/8W -> 1K
- R14: renamed from R8; moved to F.Cu
- R15: renamed from R9; moved to F.Cu
- R16: renamed from R10; moved to F.Cu
- R17: renamed from R11; moved to F.Cu
- R18: renamed from R16; moved to F.Cu
- R19: renamed from R17; moved to F.Cu
- R20: renamed from R18; moved to F.Cu
- R21: renamed from R19; moved to F.Cu
- R22: renamed from R20; moved to F.Cu
- R23: renamed from R21; moved to F.Cu
- R24: renamed from R22; moved to F.Cu
- R25: renamed from R23; moved to F.Cu
- R26: renamed from R24; moved to F.Cu
- R27: renamed from R25; moved to F.Cu
- R28: renamed from R26; moved to F.Cu
- R29: renamed from R27; moved to F.Cu
- R30: renamed from R28; moved to F.Cu
- R31: renamed from R29; moved to F.Cu
- R32: renamed from R30; moved to F.Cu
- R33: renamed from R31; moved to F.Cu
- R34: renamed from R32; moved to F.Cu
- R35: renamed from R33; moved to F.Cu
- R36: renamed from R34; moved to F.Cu
- R37: renamed from R35; moved to F.Cu
- moved TP1 101.0 mm to (106.8, 102.1), turned to 0 degrees
- moved TP3 101.0 mm to (106.8, 105.3), turned to 0 degrees
- moved TP5 101.0 mm to (106.8, 108.5), turned to 0 degrees
- moved R35 98.2 mm to (106.3, 78.5), turned to 0 degrees
- moved R28 98.2 mm to (106.4, 93.6)
- moved TP10 98.1 mm to (101.8, 73.0), turned to -90 degrees
- moved TP11 98.1 mm to (110.0, 108.5), turned to 0 degrees
- moved TP7 98.1 mm to (110.0, 102.1), turned to 0 degrees
- moved TP9 98.1 mm to (110.0, 105.3), turned to 0 degrees
- moved R34 97.5 mm to (106.3, 81.9), turned to 0 degrees
- moved R30 97.4 mm to (106.4, 94.8)
- moved R18 95.5 mm to (106.4, 87.6)
- moved R20 94.7 mm to (106.4, 88.8)
- moved R22 94.0 mm to (106.4, 90.0)
- moved TP6 93.7 mm to (101.8, 69.7), turned to -90 degrees
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- renumbered C8 to C10, C9 to C11, C10 to C12, C11 to C13, C12 to C14, C33 to C27, C34 to C28, C35 to C29, C36 to C30, C37 to C31, C38 to C32, C39 to C33, C40 to C34, C41 to C35, C42 to C36, C43 to C37, C44 to C38, C45 to C39, C46 to C40, C47 to C41, C48 to C42, C49 to C43, C51 to C45, C52 to C46, C53 to C47, C55 to C49, C56 to C50, C57 to C51, C61 to C55, C62 to C56, C66 to C60, C68 to C62, C72 to C66, C75 to C7, C76 to C8, C7 to C9, Q5 to Q3, R42 to R10, R5 to R2, R6 to R3, R36 to R38, R37 to R39, R2 to R4, R38 to R40, R39 to R5, R3 to R6, R4 to R7, R40 to R8, R41 to R9
Connections:
- C25 pad 2: +5V -> +3.3V
- C26 pad 2: +5V -> +3.3V
- C33 pad 2: Vdrive -> Vdrive_2
- C34 pad 2: Vdrive -> Vdrive_2
- C35 pad 2: Vdrive -> Vdrive_2
- C36 pad 2: Vdrive -> Vdrive_2
- C37 pad 2: Vdrive -> Vdrive_2
- C38 pad 2: Vdrive -> Vdrive_2
- C39 pad 2: Vdrive -> Vdrive_2
- C40 pad 2: Vdrive -> Vdrive_2
- C41 pad 2: Vdrive -> Vdrive_2
- C42 pad 2: Vdrive -> Vdrive_2
- C43 pad 2: Vdrive -> Vdrive_2
- C44 pad 2: Vdrive -> Vdrive_2
- C45 pad 2: Vdrive -> Vdrive_2
- C46 pad 2: Vdrive -> Vdrive_2
- C47 pad 2: Vdrive -> Vdrive_2
- C48 pad 2: Vdrive -> Vdrive_2
- C49 pad 2: Vdrive -> Vdrive_2
- C50 pad 2: Vdrive -> Vdrive_2
- C51 pad 2: Vdrive -> Vdrive_1
- C52 pad 2: Vdrive -> Vdrive_1
- C53 pad 2: Vdrive -> Vdrive_1
- C54 pad 2: Vdrive -> Vdrive_1
- C55 pad 2: Vdrive -> Vdrive_1
- C56 pad 2: Vdrive -> Vdrive_1
- C57 pad 2: Vdrive -> Vdrive_1
- C58 pad 2: Vdrive -> Vdrive_1
- C59 pad 2: Vdrive -> Vdrive_1
- C60 pad 2: Vdrive -> Vdrive_1
- C61 pad 2: Vdrive -> Vdrive_1
- C62 pad 2: Vdrive -> Vdrive_1
- C63 pad 2: Vdrive -> Vdrive_1
- C64 pad 2: Vdrive -> Vdrive_1
- C65 pad 2: Vdrive -> Vdrive_1
- C66 pad 2: Vdrive -> Vdrive_1
- C67 pad 2: Vdrive -> Vdrive_1
- C68 pad 2: Vdrive -> Vdrive_1
- J10 pad 2: Vdrive -> Vdrive_2
- J11 pad 2: Vdrive -> Vdrive_2
- J12 pad 2: Vdrive -> Vdrive_2
- J13 pad 2: Vdrive -> Vdrive_2
- J14 pad 2: Vdrive -> Vdrive_2
- J15 pad 2: Vdrive -> Vdrive_2
- J16 pad 2: Vdrive -> Vdrive_1
- J17 pad 2: Vdrive -> Vdrive_1
- J18 pad 2: Vdrive -> Vdrive_1
- J19 pad 2: Vdrive -> Vdrive_1
- J2 pad 1: +BATT -> GND
- J2 pad 2: +BATT -> GND
- J2 pad 3: GND -> VCC
- J2 pad 4: GND -> VCC
- J20 pad 2: Vdrive -> Vdrive_1
- J21 pad 2: Vdrive -> Vdrive_1
- J22 pad 2: Vdrive -> Vdrive_1
- J23 pad 2: Vdrive -> Vdrive_1
- J24 pad 2: Vdrive -> Vdrive_1
- J3 pad 1: Vdrive -> Vdrive_1
- J3 pad 2: Vdrive -> Vdrive_2
- J7 pad 2: Vdrive -> Vdrive_2
- J8 pad 2: Vdrive -> Vdrive_2
- J9 pad 2: Vdrive -> Vdrive_2
- R11 pad 1: Net-(U2-GPIO0_26) -> Net-(U2-GPIO1_3)
- R12 pad 1: BBAI_I2C_SDA -> BBAI_I2C_SCL
- R13 pad 1: BBAI_I2C_SCL -> BBAI_I2C_SDA
- SW1 pad 1: Net-(J1-Pin_1) -> unconnected-(SW1-Pad1)
- SW1 pad 3: unconnected-(SW1-Pad3) -> Net-(J1-Pin_1)
- U2 pad P8_14: Net-(U2-GPIO0_26) -> unconnected-(U2-GPIO0_26-PadP8_14)
- U2 pad P8_3: unconnected-(U2-GPIO1_6-PadP8_3) -> BBAI_ECHO
- U2 pad P8_4: unconnected-(U2-GPIO1_7-PadP8_4) -> BBAI_TRIG
- U2 pad P8_6: unconnected-(U2-GPIO1_3-PadP8_6) -> Net-(U2-GPIO1_3)
- U2 pad P9_12: BBAI_TRIG -> unconnected-(U2-GPIO1_28-PadP9_12)
- U2 pad P9_14: BBAI_PWM1A -> unconnected-(U2-GPIO1_18/PWM1A-PadP9_14)
- U2 pad P9_15: BBAI_ECHO -> unconnected-(U2-GPIO1_16-PadP9_15)
- U2 pad P9_16: unconnected-(U2-GPIO1_19/PWM1B-PadP9_16) -> BBAI_PWM1A
- U3 pad 26: PCA9685_I2C_SCL -> BBAI_I2C_SCL
- U3 pad 27: PCA9685_I2C_SDA -> BBAI_I2C_SDA
- U3 pad 28: +5V -> +3.3V
- U4 pad 26: PCA9685_I2C_SCL -> BBAI_I2C_SCL
- U4 pad 27: PCA9685_I2C_SDA -> BBAI_I2C_SDA
- U4 pad 28: +5V -> +3.3V
Routing:
- net Vdrive_1: track 0.00 -> 45.6 mm
- net +3.3V: track 0.00 -> 32.9 mm, vias 0 -> 4
- net +5V: track 0.00 -> 23.6 mm
- net HCSR04_ECHO: track 0.00 -> 14.9 mm, vias 0 -> 1
- net HCSR04_TRIG: track 0.00 -> 14.5 mm, vias 0 -> 1
- net Net-(U2-GPIO1_3): track 0.00 -> 8.30 mm
- net BBAI_TRIG: track 0.00 -> 7.13 mm
- net BBAI_ECHO: track 0.00 -> 4.30 mm
- net Net-(U4-~{OE}): track 0.00 -> 3.81 mm
- net /Servo Drivers/A1_5: track 0.00 -> 3.07 mm
- net /Servo Drivers/CH0_0: track 0.00 -> 2.75 mm
- net /Servo Drivers/CH0_7: track 0.00 -> 2.74 mm
- net /Servo Drivers/CH0_1: track 0.00 -> 2.69 mm
- net /Servo Drivers/CH0_6: track 0.00 -> 2.68 mm
- net /Servo Drivers/CH0_2: track 0.00 -> 2.62 mm
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Other:
- board size 78 x 100 mm -> 78.5 x 100 mm

Commit message: update pcb
Parts:
- moved R19 0.99 mm to (92.9, 88.1)
- moved R21 0.99 mm to (92.9, 86.9)
- moved R23 0.99 mm to (92.9, 85.7)
- moved R25 0.99 mm to (92.9, 84.5)
- moved R27 0.99 mm to (92.9, 83.2)
- moved R29 0.99 mm to (92.9, 82.0)
- moved R31 0.99 mm to (92.9, 80.8)
- moved R32 0.99 mm to (93.0, 93.8)
- moved R33 0.99 mm to (93.0, 97.3)
- moved R37 0.99 mm to (93.0, 78.5)
- moved R18 0.82 mm to (107.2, 87.6)
- moved R20 0.82 mm to (107.2, 88.8)
- moved R22 0.82 mm to (107.2, 90.0)
- moved R24 0.82 mm to (107.2, 91.2)
- moved R26 0.82 mm to (107.2, 92.4)
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Routing:
- net Net-(U3-~{OE}): track 0.00 -> 3.90 mm
- net /Servo Drivers/A0_5: track 0.00 -> 3.67 mm
- net /Servo Drivers/A0_3: track 0.00 -> 1.08 mm, vias 0 -> 1
- net /Servo Drivers/A0_4: track 0.00 -> 1.07 mm, vias 0 -> 1
- net /Servo Drivers/A1_4: track 0.00 -> 1.06 mm, vias 0 -> 1
- net /Servo Drivers/A1_3: track 0.00 -> 1.02 mm, vias 0 -> 1
- net /Servo Drivers/A1_2: track 0.00 -> 1.01 mm, vias 0 -> 1
- net /Servo Drivers/A1_1: track 0.00 -> 1.01 mm, vias 0 -> 1
- net /Servo Drivers/CH1_8: track 2.47 -> 3.46 mm
- net /Servo Drivers/CH0_7: track 2.74 -> 3.73 mm
- net /Servo Drivers/CH0_6: track 2.68 -> 3.67 mm
- net /Servo Drivers/CH0_4: track 2.55 -> 3.54 mm
- net /Servo Drivers/CH0_3: track 2.56 -> 3.55 mm
- net /Servo Drivers/CH0_2: track 2.62 -> 3.61 mm
- net /Servo Drivers/CH0_1: track 2.69 -> 3.68 mm
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
Commit message: Update PCB Ver_1.1.0
Parts:
- C31, C32: moved to F.Cu
- D4, R7: moved to B.Cu
- moved TP5 60.2 mm to (163.7, 89.0), turned to 90 degrees
- moved TP11 58.3 mm to (163.7, 85.8), turned to 90 degrees
- moved TP3 56.1 mm to (160.5, 89.0), turned to 90 degrees
- moved TP9 54.1 mm to (160.5, 85.8), turned to 90 degrees
- moved TP1 52.2 mm to (157.2, 89.0), turned to 90 degrees
- moved TP7 50.0 mm to (157.2, 85.8), turned to 90 degrees
- moved R7 24.1 mm to (107.7, 48.3)
- moved D4 24.1 mm to (111.0, 48.3)
- moved TP2 22.0 mm to (106.9, 87.9), turned to 0 degrees
- moved TP4 20.9 mm to (106.9, 85.7), turned to 0 degrees
- moved R38 19.6 mm to (73.8, 77.0), turned to 0 degrees
- moved C22 18.1 mm to (122.5, 50.9), turned to 90 degrees
- moved R39 17.7 mm to (73.7, 75.6), turned to 0 degrees
- moved R17 17.4 mm to (119.6, 48.5), turned to 0 degrees
- moved C20 16.1 mm to (121.3, 50.9), turned to 90 degrees
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Connections:
- J1 pad 1: Net-(J1-Pin_1) -> VBUS
- J2 pad 3: VCC -> VBUS
- J2 pad 4: VCC -> VBUS
- J4 pad 3: MPU6050_I2C_SCL -> BBAI_I2C_SCL
- J4 pad 4: MPU6050_I2C_SDA -> BBAI_I2C_SDA
- SW1 pad 3: Net-(J1-Pin_1) -> VBUS
Routing:
- net +5V: track 23.6 -> 170.1 mm
- net Vdrive_2: track 0.00 -> 133.3 mm, vias 0 -> 4
- net Vdrive_1: track 45.6 -> 139.5 mm, vias 0 -> 4
- net PCA_CH1_2: track 0.00 -> 68.9 mm, vias 0 -> 1
- net PCA_CH1_0: track 0.00 -> 68.1 mm, vias 0 -> 1
- net PCA_CH1_3: track 0.00 -> 67.5 mm, vias 0 -> 1
- net PCA_CH1_1: track 0.00 -> 56.3 mm, vias 0 -> 1
- net +3.3V: track 32.9 -> 87.3 mm
- net /Servo Drivers/A0_0: track 0.00 -> 26.9 mm, vias 0 -> 2
- net VCC: track 0.00 -> 25.3 mm
- net BBAI_TRIG: track 7.13 -> 31.4 mm, vias 0 -> 1
- net /Servo Drivers/A0_1: track 0.00 -> 24.2 mm, vias 0 -> 2
- net /Servo Drivers/A0_2: track 0.00 -> 21.5 mm, vias 0 -> 2
- net /Servo Drivers/A0_3: track 1.08 -> 19.1 mm, vias 1 -> 2
- net /Servo Drivers/A0_4: track 1.07 -> 16.6 mm, vias 1 -> 2
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Other:
- board size 78.5 x 100 mm -> 80.5 x 100 mm

Commit message: Update PCB
Parts:
- moved TP9 71.4 mm to (89.2, 89.8)
- moved TP11 70.2 mm to (93.6, 89.8)
- moved TP5 70.1 mm to (93.6, 87.6), turned to -90 degrees
- moved TP3 69.0 mm to (91.4, 87.6), turned to -90 degrees
- moved TP1 68.1 mm to (89.2, 87.6), turned to -90 degrees
- moved TP7 65.9 mm to (91.4, 89.8)
- moved TP12 14.4 mm to (107.0, 80.8), turned to -90 degrees
- moved TP2 6.61 mm to (111.4, 83.1), turned to 90 degrees
- moved TP10 4.74 mm to (111.4, 80.8), turned to -90 degrees
- moved R18 3.77 mm to (107.5, 88.3)
- moved R22 3.77 mm to (107.5, 90.7)
- moved R20 3.77 mm to (107.5, 89.5)
- moved R24 3.77 mm to (107.5, 91.9)
- moved R26 3.77 mm to (107.5, 93.1)
- moved R28 3.77 mm to (107.5, 94.3)
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Connections:
- TP1 pad 2: +5V -> +3.3V
- TP10 pad 2: +5V -> +3.3V
- TP11 pad 2: +5V -> +3.3V
- TP12 pad 2: +5V -> +3.3V
- TP2 pad 2: +5V -> +3.3V
- TP3 pad 2: +5V -> +3.3V
- TP4 pad 2: +5V -> +3.3V
- TP5 pad 2: +5V -> +3.3V
- TP6 pad 2: +5V -> +3.3V
- TP7 pad 2: +5V -> +3.3V
- TP8 pad 2: +5V -> +3.3V
- TP9 pad 2: +5V -> +3.3V
Routing:
- net BBAI_I2C_SCL: track 8.72 -> 187.9 mm, vias 0 -> 1
- net BBAI_I2C_SDA: track 4.18 -> 178.0 mm, vias 0 -> 1
- net +5V: track 170.1 -> 262.9 mm, vias 0 -> 2
- net PCA_CH0_5: track 0.00 -> 83.2 mm, vias 0 -> 1
- net +3.3V: track 87.3 -> 166.3 mm, vias 4 -> 12
- net PCA_CH1_4: track 0.00 -> 75.3 mm, vias 0 -> 1
- net PCA_CH0_4: track 0.00 -> 72.5 mm, vias 0 -> 1
- net Vdrive_2: track 133.3 -> 202.9 mm, vias 4 -> 10
- net PCA_CH0_6: track 0.00 -> 65.9 mm, vias 0 -> 2
- net Vdrive_1: track 139.5 -> 199.7 mm
- net PCA_CH0_0: track 0.00 -> 59.0 mm, vias 0 -> 1
- net PCA_CH1_5: track 0.00 -> 58.4 mm, vias 0 -> 2
- net PCA_CH0_7: track 0.00 -> 57.3 mm, vias 0 -> 4
- net PCA_CH0_3: track 0.00 -> 51.2 mm, vias 0 -> 1
- net PCA_CH0_8: track 0.00 -> 49.2 mm, vias 0 -> 4
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- added copper zone on F.Cu, net +3.3V
- added copper zone on F.Cu, net +5V
- added copper zone on F.Cu, net +BATT
- added copper zone on F.Cu, net Net-(D5-K)
- added copper zone on B.Cu, net VBUS
- added copper zone on F.Cu, net VCC
- added copper zone on B.Cu, net Vdrive_2
- added copper zone on F.Cu, net Vdrive_2

Commit message: update
Parts:
- moved C67 6.34 mm to (81.4, 49.6), turned to -90 degrees
- moved C63 6.25 mm to (83.1, 49.6), turned to -90 degrees
- moved R18 1.36 mm to (108.8, 88.3)
- moved R20 1.36 mm to (108.8, 89.5)
- moved R22 1.36 mm to (108.8, 90.7)
- moved R24 1.36 mm to (108.8, 91.9)
- moved R26 1.36 mm to (108.8, 93.1)
- moved R28 1.36 mm to (108.8, 94.3)
- moved R30 1.36 mm to (108.8, 95.6)
- moved R36 1.36 mm to (108.8, 98.0)
- moved C55 1.04 mm to (68.0, 49.6)
- moved C60 1.04 mm to (66.3, 49.6)
- moved C61 1.04 mm to (68.0, 49.6)
- moved C65 1.04 mm to (66.3, 49.6)
Routing:
- net Vdrive_1: track 199.7 -> 256.0 mm, vias 4 -> 13
- net +5V: track 262.9 -> 277.4 mm, vias 2 -> 5
- net Vdrive_2: track 202.9 -> 214.4 mm, vias 10 -> 11
- net PCA_CH1_5: track 58.4 -> 63.5 mm
- net PCA_CH1_8: track 23.9 -> 27.6 mm
- net PCA_CH1_4: track 75.3 -> 71.8 mm
- net PCA_CH1_7: track 32.5 -> 35.4 mm
- net +3.3V: track 166.3 -> 164.2 mm, vias 12 -> 11
- net BBAI_I2C_SDA: track 178.0 -> 180.1 mm
- net BBAI_I2C_SCL: track 187.9 -> 189.9 mm
- net PCA_CH0_1: track 46.6 -> 44.6 mm
- net GND: track 4.77 -> 6.48 mm, vias 0 -> 1
- net PCA_CH0_0: track 59.0 -> 57.7 mm
- net Net-(U3-~{OE}): track 4.09 -> 5.45 mm
- net /Servo Drivers/A0_5: track 18.0 -> 19.4 mm
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- added copper zone on B.Cu, net GND
- added copper zone on F.Cu, net GND
- added copper zone on B.Cu, net Vdrive_1
- added copper zone on F.Cu, net Vdrive_1

Commit message: Update PCB_Ver1.1.0
Parts:
- moved C44 2.05 mm to (111.2, 132.9)
- moved C48 2.05 mm to (111.2, 134.7)
- moved J13 2.05 mm to (112.1, 139.0)
- moved D4 0.15 mm to (111.0, 48.4)
- moved R7 0.15 mm to (107.7, 48.4)
- moved C10 0.15 mm to (73.4, 60.3)
- moved C11 0.15 mm to (75.6, 65.8)
- moved C12 0.15 mm to (75.6, 60.3)
- moved C13 0.15 mm to (73.4, 65.8)
- moved C14 0.15 mm to (77.8, 60.3)
- moved C9 0.15 mm to (77.8, 65.8)
Routing:
- net GND: track 6.48 -> 20.7 mm, vias 1 -> 238
- net +3.3V: track 164.2 -> 174.1 mm, vias 11 -> 12
- net Vdrive_1: track 256.0 -> 262.7 mm, vias 13 -> 14
- net Vdrive_2: track 214.4 -> 219.6 mm, vias 11 -> 12
- net PCA_CH0_6: track 67.3 -> 69.8 mm
- net PCA_CH0_1: track 44.6 -> 46.9 mm
- net PCA_CH0_0: track 57.7 -> 59.8 mm
- net BBAI_PWM1A: track 0.00 -> 2.01 mm
- net /Servo Drivers/A1_5: track 16.5 -> 18.5 mm
- net PCA_CH1_4: track 71.8 -> 73.3 mm
- net BBAI_I2C_SDA: track 180.1 -> 178.6 mm
- net BBAI_I2C_SCL: track 189.9 -> 188.6 mm
- net PCA_CH1_2: track 77.3 -> 78.2 mm
- net PCA_CH1_3: track 70.8 -> 71.6 mm
- net PCA_CH0_4: track 71.5 -> 72.2 mm
Other:
- board text added: "+"
- board text added: "5V"
- board text added: "A0"
- board text added: "A1"
- board text added: "A2"
- board text added: "A3"
- board text added: "A4"
- board text added: "A5"
- board text added: "C0_0"
- board text added: "C0_1"
- board text added: "C0_2"
- board text added: "C0_3"
- board text added: "C0_4"
- board text added: "C0_5"
- board text added: "CH1_0"
- board text added: "CH1_1"
- board text added: "CH1_2"
- board text added: "CH1_3"
- board text added: "CH1_4"
- board text added: "CH1_5"
- board text added: "CH1_7"
- board text added: "CH1_8"
- board text added: "ECHO"
- board text added: "GND"
- board text added: "TRIG"
- board text added: "VBUS"
- board text added: "VDRIVE"

Commit message: update pcb
Parts:
- moved J24 0.07 mm to (104.1, 55.0)
Routing:
- net GND: track 20.7 -> 43.0 mm, vias 238 -> 529
- net +5V: track 277.4 -> 267.1 mm
- net Vdrive_2: track 219.6 -> 223.7 mm
- net VCC: track 28.0 -> 25.3 mm
- net BBAI_I2C_SCL: track 188.6 -> 187.1 mm
- net PCA_CH1_3: track 71.6 -> 72.5 mm
- net /Servo Drivers/A1_4: track 20.4 -> 21.2 mm
- net PCA_CH1_7: track 35.4 -> 34.6 mm
- net PCA_CH1_4: track 73.3 -> 74.1 mm
- net /Servo Drivers/A1_3: track 17.4 -> 18.1 mm
- net PCA_CH1_6: track 39.6 -> 39.0 mm
- net PCA_CH0_6: track 69.8 -> 69.3 mm
- net (no net): vias 3 -> 0
