File: hardware/Source/Ver_1.1.0/BBAI.kicad_sch (KiCad schematic)
At the start: 0 parts

Commit message: update folder hardware
Parts:
- added C1, C3: 10uF/16V, automative_hexapod:Ceramic_Cap_0805, symbol automative_hexapod:Ceramic_Cap_0805_10uF_16V
- added C2, C4: 100nF/50V, automative_hexapod:Ceramic_Cap_0805, symbol automative_hexapod:Ceramic_Cap_0805_100nF_50V
- added D1: LED_0805, automative_hexapod:LED_0805, symbol automative_hexapod:LED_0805
- added R18: 1K/1%/1/8W, automative_hexapod:Res_0805, symbol automative_hexapod:Res_1K_0805_1%
- added U1: ~, automative_hexapod:BeagleBone_AI, symbol automative_hexapod:BeagleBone_AI
Connections:
- new net: R18.1, U1.P8_14 (GPIO0_26)
- new net: D1.2 (A), R18.2
- new net +3.3V: C3.2, C4.2, U1.P9_3 (3V3), U1.P9_4 (3V3)
- new net +5V: C1.2, C2.2, U1.P9_5 (5V_RAW), U1.P9_6 (5V_RAW)
- new net BBAI_ECHO: U1.P9_15 (GPIO1_16)
- new net BBAI_I2C_SCL: U1.P9_19 (I2C2_SCL/GPIO0_13)
- new net BBAI_I2C_SDA: U1.P9_20 (I2C2_SDA/GPIO0_12)
- new net BBAI_PWM1A: U1.P9_14 (GPIO1_18/PWM1A)
- new net BBAI_TRIG: U1.P9_12 (GPIO1_28)
- new net GND: C1.1, C2.1, C3.1, C4.1, D1.1 (K), U1.P8_1 (GND), U1.P8_2 (GND), U1.P9_1 (GND), U1.P9_2 (GND)
- no-connect marks 0 -> 78

Commit message: Update Library for Ver 2
Parts:
- removed C1, C3: 10uF/16V, automative_hexapod:Ceramic_Cap_0805, symbol automative_hexapod:Ceramic_Cap_0805_10uF_16V
- removed C2, C4: 100nF/50V, automative_hexapod:Ceramic_Cap_0805, symbol automative_hexapod:Ceramic_Cap_0805_100nF_50V
- added C10, C8: 22uF, automative_hexapod:Ceramic_Cap_1206, symbol automative_hexapod:Ceramic_Cap_1206_22uF_10V
- added C11, C12: 100nF, automative_hexapod:Ceramic_Cap_0805, symbol automative_hexapod:Ceramic_Cap_0805_100nF_50V
- added C7, C9: 22uF, automative_hexapod:Ceramic_Cap_1206, symbol automative_hexapod:Ceramic_Cap_1206_22uF_25V
- D5: renamed from D1; Supply Name (none) -> Thegioiic; Supply Part Number (none) -> LED Xanh Lá 0805 Dán SMD Trong Suốt; Supply name Thegioiic -> (none); Supply part number LED Xanh Lá 0805 Dán SMD Trong Suốt -> (none)
- R6: renamed from R18; Supply Name (none) -> thegioiic; Supply Part Number (none) -> Điện Trở 1 KOhm 0805 1%; Supply name thegioiic -> (none); Supply part number Điện Trở 1 KOhm 0805 1% -> (none)
- renumbered U1 to U2
Connections:
- net +3.3V: now also C10.2, C12.2, C8.2
- net +5V: now also C11.2, C7.2, C9.2
- net GND: now also C10.1, C11.1, C12.1, C7.1, C8.1, C9.1
Other:
- title: (none) -> BBAI
