File: hardware/Source/Ver_1.1.0/BBAI.kicad_sch (KiCad schematic)
At the start: 7 parts

Commit message: update pcb v1.1.0
Parts:
- removed C1, C3: 10uF/16V, automative_hexapod:Ceramic_Cap_0805, symbol automative_hexapod:Ceramic_Cap_0805_10uF_16V
- removed C2, C4: 100nF/50V, automative_hexapod:Ceramic_Cap_0805, symbol automative_hexapod:Ceramic_Cap_0805_100nF_50V
- added C10, C8: 22uF, automative_hexapod:Ceramic_Cap_1206, symbol automative_hexapod:Ceramic_Cap_1206_22uF_10V
- added C11, C12: 100nF, automative_hexapod:Ceramic_Cap_1206, symbol automative_hexapod:Ceramic_Cap_1206_100nF_50V
- added C7, C9: 22uF, automative_hexapod:Ceramic_Cap_1206, symbol automative_hexapod:Ceramic_Cap_1206_22uF_25V
- D6: renamed from D1; Supply Name (none) -> Thegioiic; Supply Part Number (none) -> LED Xanh Lá 0805 Dán SMD Trong Suốt; Supply URL https://www.thegioiic.com/led-xanh-la-0805-dan-smd-trong-su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 -> https://www.Thegioiic.com/led-xanh-la-0805-dan-smd-trong-su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; Supply name Thegioiic -> (none); Supply part number LED Xanh Lá 0805 Dán SMD Trong Suốt -> (none)
- R7: renamed from R18; value 1K/1%/1/8W -> 1K; Supply Name (none) -> Thegioiic; Supply Part Number (none) -> Điện Trở 1 KOhm 0805 1%; Supply URL https://www.thegioiic.com/dien-tro-1-kohm-0805-1- -> https://www.Thegioiic.com/dien-tro-1-kohm-0805-1-; Supply name thegioiic -> (none); Supply part number Điện Trở 1 KOhm 0805 1% -> (none); Value 2 (none) -> 1/8W; Value 3 (none) -> 0805; Value 4 (none) -> 1%
- renumbered U1 to U2
Connections:
- net +3.3V: now also C10.2, C12.1, C8.2
- net +5V: now also C11.1, C7.2, C9.2
- net GND: now also C10.1, C11.2, C12.2, C7.1, C8.1, C9.1
Other:
- title: (none) -> BBAI

Commit message: update pcb and schematic
Parts:
- added R12, R13: 10kOhm, automative_hexapod:Res_0603, symbol automative_hexapod:Res_10K_0603_1%
- renumbered C8 to C10, C9 to C11, C10 to C12, C11 to C13, C12 to C14, C7 to C9, R7 to R11
Connections:
- net +3.3V: now also R12.2, R13.2
- net BBAI_ECHO: now also U2.P8_3 (GPIO1_6); no longer U2.P9_15 (GPIO1_16)
- net BBAI_I2C_SCL: now also R12.1
- net BBAI_I2C_SDA: now also R13.1
- net BBAI_PWM1A: now also U2.P9_16 (GPIO1_19/PWM1B); no longer U2.P9_14 (GPIO1_18/PWM1A)
- net BBAI_TRIG: now also U2.P8_4 (GPIO1_7); no longer U2.P9_12 (GPIO1_28)
- net at R11.1: now also U2.P8_6 (GPIO1_3); no longer U2.P8_14 (GPIO0_26)
Other:
- moved on the sheet: D6, R11
