File: hardware/Source/Ver_1.1.0/HC-SR04.kicad_sch (KiCad schematic)
At the start: 0 parts

Commit message: Update Library for Ver 2
Parts:
- added C33: 10uF, automative_hexapod:Ceramic_Cap_0805, symbol automative_hexapod:Ceramic_Cap_0805_10uF_16V
- added C34: 100nF, automative_hexapod:Ceramic_Cap_0805, symbol automative_hexapod:Ceramic_Cap_0805_100nF_50V
- added J6: Connector, automative_hexapod:JST-XH-SMD-4-2.54mm, symbol automative_hexapod:JST-XH-SMD-4-2.54mm
Connections:
- new net +5V: C33.2, C34.2
- new net GND: C33.1, C34.1
Other:
- title: (none) -> HC-SR04
