File: hardware/Source/Ver_1.1.0/IMU.kicad_sch (KiCad schematic)
At the start: 0 parts

Commit message: Update Library for Ver 2
Parts:
- added C31: 10uF, automative_hexapod:Ceramic_Cap_0805, symbol automative_hexapod:Ceramic_Cap_0805_10uF_16V
- added C32: 100nF, automative_hexapod:Ceramic_Cap_0805, symbol automative_hexapod:Ceramic_Cap_0805_100nF_50V
- added J4: MPU6050, automative_hexapod:MPU6050, symbol automative_hexapod:MPU6050
Connections:
- new net +5V: C31.2, C32.2, J4.1 (Pin_1)
- new net GND: C31.1, C32.1, J4.2 (Pin_2)
- new net MPU6050_I2C_SCL: J4.3 (Pin_3)
- new net MPU6050_I2C_SDA: J4.4 (Pin_4)
- no-connect marks 0 -> 4
Other:
- title: (none) -> IMU
