File: hardware/Source/Ver_1.1.0/PowerSupply.kicad_sch (KiCad schematic)
At the start: 9 parts, among them U2 XL4005E1

Commit message: Update Library for Ver 2
Parts:
- removed C29: 330uF/50V, Capacitor_SMD:CP_Elec_10x10.5, symbol automative_hexapod:Cap_Polarized_SMD_330uF_50V
- removed C38: 220uF/50V, Capacitor_SMD:CP_Elec_10x10.5, symbol automative_hexapod:Cap_Polarized_SMD_220uF_50V
- removed C45, C46: 1uF/16V, automative_hexapod:Ceramic_Cap_0805, symbol automative_hexapod:Ceramic_Cap_0805_1uF_16V
- removed R13: 10.5K/1%/1/8W, automative_hexapod:Res_0805, symbol automative_hexapod:Res_10.5K_0805_1%
- removed R14: 2K/1%/1/8W, automative_hexapod:Res_0805, symbol automative_hexapod:Res_2K_0805_1%
- added C1, C2: 220uF, Capacitor_SMD:CP_Elec_10x10.5, symbol automative_hexapod:Cap_Polarized_SMD_220uF_50V
- added C3, C4: 1uF, automative_hexapod:Ceramic_Cap_1206, symbol automative_hexapod:Ceramic_Cap_1206_1uF_50V
- added C5, C6: 330uF, Capacitor_SMD:CP_Elec_10x10.5, symbol automative_hexapod:Cap_Polarized_SMD_330uF_50V
- added D1: PIN, automative_hexapod:LED_0805, symbol automative_hexapod:LED_0805
- added D2: 5V, automative_hexapod:LED_0805, symbol automative_hexapod:LED_0805
- added D3: 3.3V, automative_hexapod:LED_0805, symbol automative_hexapod:LED_0805
- added F1: Fuse, automative_hexapod:FUSE_SMD_1808, symbol automative_hexapod:Fuse_1808
- added J1: Pin Connector, automative_hexapod:Connector-Pin, symbol automative_hexapod:Pin Connector
- added J2, J3: Connector, automative_hexapod:TerminalBlock_Phoenix_MKDS-1,5-4-5.08_1x04_P5.08mm_Horizontal, symbol automative_hexapod:KF120-4-V Domino
- added R1, R4: 10.5kOhm, automative_hexapod:Res_0805, symbol automative_hexapod:Res_10.5K_0805_1%
- added R2: 5.6kOhm, automative_hexapod:Res_0805, symbol automative_hexapod:Res_5.6K_0805_1%
- added R3, R5: 2kOhm, automative_hexapod:Res_0805, symbol automative_hexapod:Res_2K_0805_1%
- added SW1: MTS-103, automative_hexapod:MTS-103_JCV, symbol automative_hexapod:MTS-103
- L1: Supply Name ThegioiIC -> Thegioiic
- renumbered D2 to D4, U2 to U1
Connections:
- net +5V: now also C4.2, C5.1, C6.1, D2.2 (A), R4.2
- net GND: now also C1.2, C2.2, C3.1, C4.1, C5.2, C6.2, R1.1, R2.1, R3.1, R5.1
- net VCC: now also C1.1, C2.1, C3.2, D1.2 (A)
- net at U1.2 (FB): now also R4.1, R5.2
- new net: D3.1 (K), R3.2
- new net: D2.1 (K), R2.2
- new net: D1.1 (K), R1.2
- new net +3.3V: D3.2 (A)
Other:
- title: (none) -> Power Supply
- moved on the sheet: D4, L1, U1
