File: hardware/Source/Ver_1.1.0/PowerSupply.kicad_sch (KiCad schematic)
At the start: 0 parts

Commit message: update folder hardware
Parts:
- added C29: 330uF/50V, Capacitor_SMD:CP_Elec_10x10.5, symbol automative_hexapod:Cap_Polarized_SMD_330uF_50V
- added C38: 220uF/50V, Capacitor_SMD:CP_Elec_10x10.5, symbol automative_hexapod:Cap_Polarized_SMD_220uF_50V
- added C45, C46: 1uF/16V, automative_hexapod:Ceramic_Cap_0805, symbol automative_hexapod:Ceramic_Cap_0805_1uF_16V
- added D2: MBR20100CT, automative_hexapod:TO-220-3, symbol automative_hexapod:MBR20100CT
- added L1: 27uH 5.7A, automative_hexapod:IND_CDRH127_LDNP-470MC_SUM, symbol automative_hexapod:CDRH127_1280-270_ 27uH-5.7A
- added R13: 10.5K/1%/1/8W, automative_hexapod:Res_0805, symbol automative_hexapod:Res_10.5K_0805_1%
- added R14: 2K/1%/1/8W, automative_hexapod:Res_0805, symbol automative_hexapod:Res_2K_0805_1%
- added U2: XL4005E1, automative_hexapod:TO-263-5, symbol automative_hexapod:XL4005E1
Connections:
- new net: D2.2, L1.1, U2.3 (SW)
- new net: R13.1, R14.2, U2.2 (FB)
- new net +5V: C29.1, C46.2, L1.2, R13.2
- new net GND: C29.2, C38.2, C45.1, C46.1, D2.1, R14.1, U2.1 (GND)
- new net VCC: C38.1, C45.2, U2.4 (EN), U2.5 (VIN)
- no-connect marks 0 -> 1

Commit message: update pcb v1.1.0
Parts:
- removed C29: 330uF/50V, Capacitor_SMD:CP_Elec_10x10.5, symbol automative_hexapod:Cap_Polarized_SMD_330uF_50V
- removed C38: 220uF/50V, Capacitor_SMD:CP_Elec_10x10.5, symbol automative_hexapod:Cap_Polarized_SMD_220uF_50V
- removed C45, C46: 1uF/16V, automative_hexapod:Ceramic_Cap_0805, symbol automative_hexapod:Ceramic_Cap_0805_1uF_16V
- removed D2: MBR20100CT, automative_hexapod:TO-220-3, symbol automative_hexapod:MBR20100CT
- removed L1: 27uH 5.7A, automative_hexapod:IND_CDRH127_LDNP-470MC_SUM, symbol automative_hexapod:CDRH127_1280-270_ 27uH-5.7A
- removed R13: 10.5K/1%/1/8W, automative_hexapod:Res_0805, symbol automative_hexapod:Res_10.5K_0805_1%
- removed R14: 2K/1%/1/8W, automative_hexapod:Res_0805, symbol automative_hexapod:Res_2K_0805_1%
- removed U2: XL4005E1, automative_hexapod:TO-263-5, symbol automative_hexapod:XL4005E1
- added C1: 100uF, automative_hexapod:CP_Elec_6.3x5.4, symbol automative_hexapod:Cap_Polarized_SMD_100uF_35V
- added C2: 100nF, automative_hexapod:Ceramic_Cap_1206, symbol automative_hexapod:Ceramic_Cap_1206_100nF_50V
- added C3: 4.7nF, automative_hexapod:Ceramic_Cap_0603, symbol automative_hexapod:Ceramic_Cap_0603_4.7nF_50V
- added C4: 39pF, automative_hexapod:Ceramic_Cap_0603, symbol automative_hexapod:Ceramic_Cap_0603_39pF_50V
- added C5: 10nF, automative_hexapod:Ceramic_Cap_0603, symbol automative_hexapod:Ceramic_Cap_0603_10nF_50V
- added C6: 100nF, automative_hexapod:Ceramic_Cap_0603, symbol automative_hexapod:Ceramic_Cap_0603_100nF_50V
- added C75, C76: 47uF, automative_hexapod:Ceramic_Cap_1206, symbol automative_hexapod:Ceramic_Cap_1206_47uF_16V
- added D1, D2: PIN, automative_hexapod:LED_0805, symbol automative_hexapod:LED_0805
- added D3: 5V, automative_hexapod:LED_0805, symbol automative_hexapod:LED_0805
- added D4: 3.3V, automative_hexapod:LED_0805, symbol automative_hexapod:LED_0805
- added D5: SS54, automative_hexapod:D_SMA, symbol automative_hexapod:SS54
- added F1: Fuse, automative_hexapod:FUSE_SMD_1808, symbol automative_hexapod:Fuse_1808
- added J1: Pin Connector, automative_hexapod:Connector-Pin, symbol automative_hexapod:Pin Connector
- added J2, J3: Connector, automative_hexapod:TerminalBlock_Phoenix_MKDS-1,5-4-5.08_1x04_P5.08mm_Horizontal, symbol automative_hexapod:KF120-4-V Domino
- added L1: 10uH 4A, automative_hexapod:Inductor_0630, symbol automative_hexapod:0630_10uH-4A
- added R1, R2: 10.5kOhm, automative_hexapod:Res_0805, symbol automative_hexapod:Res_10.5K_0805_1%
- added R3: 5.6kOhm, automative_hexapod:Res_0805, symbol automative_hexapod:Res_5.6K_0805_1%
- added R39: 30kOhm, automative_hexapod:Res_0603, symbol automative_hexapod:Res_30K_0603_1%
- added R4: 2kOhm, automative_hexapod:Res_0805, symbol automative_hexapod:Res_2K_0805_1%
- added R40: 2.49kOhm, automative_hexapod:Res_0603, symbol automative_hexapod:Res_2.49K_0603_1%
- added R41: 49.9kOhm, automative_hexapod:Res_0603, symbol automative_hexapod:Res_49.9K_0603_1%
- added R42: 10kOhm, automative_hexapod:Res_0603, symbol automative_hexapod:Res_10K_0603_1%
- added R5: 100kOhm, automative_hexapod:Res_0603, symbol automative_hexapod:Res_100K_0603_1%
- added R6: 20kOhm, automative_hexapod:Res_0603, symbol automative_hexapod:Res_20K_0603_1%
- added SW1: MTS-102-C3, automative_hexapod:MTS-102-C3, symbol automative_hexapod:MTS-102-C3
- added U1: TPS54331DR, automative_hexapod:SOIC-8, symbol automative_hexapod:TPS54331DR
Connections:
- net +5V: now also C75.2, C76.2, D3.2 (A), L1.2, R40.2
- net GND: now also C1.2, C2.2, C4.1, C5.1, C75.1, C76.1, D5.1 (A), J1.2 (Pin_2), J2.3 (Pin_3), J2.4 (Pin_4), J3.3 (Pin_3), J3.4 (Pin_4), R1.1, R2.1, R3.1, R39.1, R4.1, R42.1, R6.1, SW1.SH, U1.7 (GND)
- net VCC: now also C1.1, C2.1, D2.2 (A), F1.1, R5.2, U1.2 (VIN)
- new net: D4.1 (K), R4.2
- new net: D1.1 (K), R1.2
- new net: C6.2, D5.2 (K), L1.1, U1.8 (PH)
- new net: D3.1 (K), R3.2
- new net: R41.1, R42.2, U1.5 (VSENSE)
- new net: R40.1, R41.2
- new net: J1.1 (Pin_1), SW1.1
- new net: R5.1, R6.2, U1.3 (EN)
- new net: C6.1, U1.1 (BOOT)
- new net: C5.2, U1.4 (SS)
- new net: C3.2, C4.2, U1.6 (COMP)
- new net: D2.1 (K), R2.2
- new net: C3.1, R39.2
- new net +3.3V: D4.2 (A)
- new net +BATT: D1.2 (A), F1.2, J2.1 (Pin_1), J2.2 (Pin_2), SW1.2
- new net Vdrive: J3.1 (Pin_1), J3.2 (Pin_2)
Other:
- title: (none) -> Power Supply

Commit message: update pcb and schematic
Parts:
- renumbered C75 to C7, C76 to C8, R42 to R10, R5 to R2, R6 to R3, R2 to R4, R39 to R5, R3 to R6, R4 to R7, R40 to R8, R41 to R9
Connections:
- net +BATT: no longer J2.1 (Pin_1), J2.2 (Pin_2)
- net GND: now also J2.1 (Pin_1), J2.2 (Pin_2); no longer J2.3 (Pin_3), J2.4 (Pin_4)
- net VCC: now also J2.3 (Pin_3), J2.4 (Pin_4)
- net at J1.1 (Pin_1): now also SW1.3; no longer SW1.1
- net Vdrive renamed Vdrive_1
- net Vdrive_1: no longer J3.2 (Pin_2)
- new net Vdrive_2: J3.2 (Pin_2)
Other:
- moved on the sheet: J1

Commit message: Update PCB Ver_1.1.0
Connections:
- net VCC: no longer J2.3 (Pin_3), J2.4 (Pin_4)
- net VBUS: now reaches J1.1 (Pin_1), SW1.3
- net VBUS: now also J2.3 (Pin_3), J2.4 (Pin_4)
Other:
- moved on the sheet: J1
Changed lines of the file:
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@@
 	)
 	(junction
+		(at 186.69 128.27)
+		(diameter 0)
+		(color 0 0 0 0)
+	)
+	(junction
 		(at 163.83 38.1)
 		(diameter 0)
@@
 	(wire
 		(pts
+			(xy 186.69 128.27) (xy 200.66 128.27)
+		)
+		(stroke
+			(width 0)
+			(type default)
+		)
+	)
+	(wire
+		(pts
 			(xy 236.22 116.84) (xy 236.22 114.3)
 		)
@@
 	(wire
 		(pts
+			(xy 186.69 124.46) (xy 186.69 128.27)
+		)
+		(stroke
+			(width 0)
+			(type default)
+		)
+	)
+	(wire
+		(pts
 			(xy 25.4 30.48) (xy 25.4 33.02)
 		)
@@
 	(wire
 		(pts
-			(xy 194.31 133.35) (xy 194.31 130.81)
+			(xy 187.96 133.35) (xy 187.96 130.81)
 		)
 		(stroke
@@
 	(wire
 		(pts
-			(xy 189.23 128.27) (xy 200.66 128.27)
+			(xy 181.61 128.27) (xy 186.69 128.27)
 		)
 		(stroke
@@
 	(wire
 		(pts
-			(xy 194.31 130.81) (xy 189.23 130.81)
+			(xy 187.96 130.81) (xy 181.61 130.81)
 		)
 		(stroke
@@
 	)
 	(symbol
+		(lib_id "power:VBUS")
+		(at 186.69 124.46 0)
+		(unit 1)
+		(exclude_from_sim no)
+		(in_bom yes)
+		(on_board yes)
+		(dnp no)
+		(fields_autoplaced yes)
+		(property "Reference" "#PWR0186"
+			(at 186.69 128.27 0)
+			(effects
+				(font
+					(size 1.27 1.27)
+				)
+				(hide yes)
+			)
+		)
+		(property "Value" "VBUS"
+			(at 186.69 119.38 0)
+			(effects
+				(font
+					(size 1.27 1.27)
+				)
+			)
+		)
+		(property "Footprint" ""
+			(at 186.69 124.46 0)
+			(effects
+				(font
+					(size 1.27 1.27)
+				)
+				(hide yes)
+			)
+		)
+		(property "Datasheet" ""
+			(at 186.69 124.46 0)
+			(effects
+				(font
+					(size 1.27 1.27)
+				)
+				(hide yes)
+			)
+		)
+		(property "Description" "Power symbol creates a global label with name \"VBUS\""
+			(at 186.69 124.46 0)
+			(effects
+				(font
+					(size 1.27 1.27)
+				)
+				(hide yes)
+			)
+		)
+		(pin "1"
+		)
+		(instances
+			(project "Automative_Hexapod"
+				(path "/c07b6013-2147-4cef-a16e-342deb9ccbf5/e9a15bf3-25b5-4588-8308-b7d586974115"
+					(reference "#PWR0186")
+					(unit 1)
+				)
+			)
+		)
+	)
+	(symbol
 		(lib_id "power:GND")
 		(at 101.6 35.56 270)
@@
 	(symbol
 		(lib_id "automative_hexapod:Pin Connector")
-		(at 184.15 128.27 0)
+		(at 176.53 128.27 0)
 		(mirror y)
 		(unit 1)
@@
 		(dnp no)
 		(property "Reference" "J1"
-			(at 182.88 126.9999 0)
+			(at 175.26 126.9999 0)
 			(effects
 				(font
@@
 		)
 		(property "Value" "Pin Connector"
-			(at 182.88 129.5399 0)
+			(at 175.26 129.5399 0)
 			(effects
 				(font
@@
 		)
 		(property "Footprint" "automative_hexapod:Connector-Pin"
-			(at 183.388 137.16 0)
+			(at 175.768 137.16 0)
 			(effects
 				(font
@@
 		)
 		(property "Datasheet" "~"
-			(at 184.15 128.27 0)
+			(at 176.53 128.27 0)
 			(effects
 				(font
@@
 		)
 		(property "Description" "~"
-			(at 182.118 137.16 0)
+			(at 174.498 137.16 0)
 			(effects
 				(font
@@
 		)
 		(property "Value 2" "~"
-			(at 182.88 131.445 0)
+			(at 175.26 131.445 0)
 			(effects
 				(font
@@
 		)
 		(property "Value 3" "~"
-			(at 182.88 132.715 0)
+			(at 175.26 132.715 0)
 			(effects
 				(font
@@
 		)
 		(property "Value 4" "~"
-			(at 184.15 128.27 0)
+			(at 176.53 128.27 0)
 			(effects
 				(font
@@
 		)
 		(property "Supply Name" "~"
-			(at 182.118 137.16 0)
+			(at 174.498 137.16 0)
 			(effects
 				(font
@@
 		)
 		(property "Supply Part Number" "~"
-			(at 184.15 137.16 0)
+			(at 176.53 137.16 0)
 			(effects
 				(font
@@
 		)
 		(property "Supply URL" "~"
-			(at 184.15 137.16 0)
+			(at 176.53 137.16 0)
 			(effects
 				(font
@@
 	(symbol
 		(lib_id "power:GND")
-		(at 194.31 133.35 0)
+		(at 187.96 133.35 0)
 		(unit 1)
 		(exclude_from_sim no)
@@
 		(fields_autoplaced yes)
 		(property "Reference" "#PWR017"
-			(at 194.31 139.7 0)
+			(at 187.96 139.7 0)
 			(effects
 				(font
@@
 		)
 		(property "Value" "GND"
-			(at 194.31 138.43 0)
+			(at 187.96 138.43 0)
 			(effects
 				(font
@@
 		)
 		(property "Footprint" ""
-			(at 194.31 133.35 0)
+			(at 187.96 133.35 0)
 			(effects
 				(font
@@
 		)
 		(property "Datasheet" ""
-			(at 194.31 133.35 0)
+			(at 187.96 133.35 0)
 			(effects
 				(font
@@
 		)
 		(property "Description" "Power symbol creates a global label with name \"GND\" , ground"
-			(at 194.31 133.35 0)
+			(at 187.96 133.35 0)
 			(effects
 				(font
@@
 	)
 	(symbol
-		(lib_id "power:VCC")
-		(at 236.22 107.95 0)
-		(unit 1)
-		(exclude_from_sim no)
-		(in_bom yes)
-		(on_board yes)
-		(dnp no)
-		(fields_autoplaced yes)
-		(property "Reference" "#PWR022"
-			(at 236.22 111.76 0)
-			(effects
-				(font
-					(size 1.27 1.27)
-				)
-				(hide yes)
-			)
-		)
-		(property "Value" "VCC"
-			(at 236.22 102.87 0)
-			(effects
-				(font
-					(size 1.27 1.27)
-				)
-			)
-		)
-		(property "Footprint" ""
-			(at 236.22 107.95 0)
-			(effects
-				(font
-					(size 1.27 1.27)
-				)
-				(hide yes)
-			)
-		)
-		(property "Datasheet" ""
-			(at 236.22 107.95 0)
-			(effects
-				(font
-					(size 1.27 1.27)
-				)
-				(hide yes)
-			)
-		)
-		(property "Description" "Power symbol creates a global label with name \"VCC\""
-			(at 236.22 107.95 0)
-			(effects
-				(font
-					(size 1.27 1.27)
-				)
-				(hide yes)
-			)
-		)
-		(pin "1"
-		)
-		(instances
-			(project "Automative_Hexapod"
-				(path "/c07b6013-2147-4cef-a16e-342deb9ccbf5/e9a15bf3-25b5-4588-8308-b7d586974115"
-					(reference "#PWR022")
-					(unit 1)
-				)
-			)
-		)
-	)
-	(symbol
 		(lib_id "automative_hexapod:Fuse_1808")
 		(at 191.77 114.3 0)
@@
 					(unit 1)
 				)
+			)
+		)
+	)
+	(symbol
+		(lib_id "power:VBUS")
+		(at 236.22 107.95 0)
+		(unit 1)
+		(exclude_from_sim no)
+		(in_bom yes)
+		(on_board yes)
+		(dnp no)
+		(fields_autoplaced yes)
+		(property "Reference" "#PWR0187"
+			(at 236.22 111.76 0)
+			(effects
+				(font
+					(size 1.27 1.27)
+				)
+				(hide yes)
+			)
+		)
+		(property "Value" "VBUS"
+			(at 236.22 102.87 0)
+			(effects
+				(font
+					(size 1.27 1.27)
+				)
+			)
+		)
+		(property "Footprint" ""
+			(at 236.22 107.95 0)
+			(effects
+				(font
+					(size 1.27 1.27)
+				)
+				(hide yes)
+			)
+		)
+		(property "Datasheet" ""
+			(at 236.22 107.95 0)
+			(effects
+				(font
+					(size 1.27 1.27)
+				)
+				(hide yes)
+			)
+		)
+		(property "Description" "Power symbol creates a global label with name \"VBUS\""
+			(at 236.22 107.95 0)
+			(effects
+				(font
+					(size 1.27 1.27)
+				)
+				(hide yes)
+			)
+		)
+		(pin "1"
+		)
+		(instances
+			(project "Automative_Hexapod"
+				(path "/c07b6013-2147-4cef-a16e-342deb9ccbf5/e9a15bf3-25b5-4588-8308-b7d586974115"
+					(reference "#PWR0187")
+					(unit 1)
+				)
