File: hardware/Source/Ver_1.1.0/ServoDrivers.kicad_sch (KiCad schematic)
At the start: 0 parts

Commit message: Update Library for Ver 2
Parts:
- added C29: 10uF, automative_hexapod:Ceramic_Cap_0805, symbol automative_hexapod:Ceramic_Cap_0805_10uF_16V
- added C30: 100nF, automative_hexapod:Ceramic_Cap_0805, symbol automative_hexapod:Ceramic_Cap_0805_100nF_50V
- added R15, R16, R17, R18, R19, R20, R21: 10kOhm, automative_hexapod:Res_0603, symbol automative_hexapod:Res_10K_0603_1%
- added R22, R23, R24, R25: 220Ohm, automative_hexapod:R_Array_Convex_4x0603, symbol automative_hexapod:Res_220_4D03_5%
- added TP1, TP2, TP3, TP4, TP5, TP6: ~, automative_hexapod:SolderBridgeOpen, symbol automative_hexapod:Jumper_Open
- added U3: PCA9685PW, automative_hexapod:TSSOP-28_4.4x9.7mm_P0.65mm, symbol automative_hexapod:PCA9685PW
Connections:
- new net: R21.2, U3.23 (~{OE})
- new net +5V: C29.2, C30.2, TP1.2, TP2.2, TP3.2, TP4.2, TP5.2, TP6.2, U3.28 (VDD)
- new net A0_0: R15.2, TP1.1, U3.1 (A0)
- new net A1_0: R16.2, TP2.1, U3.2 (A1)
- new net A2_0: R17.2, TP3.1, U3.3 (A2)
- new net A3_0: R18.2, TP4.1, U3.4 (A3)
- new net A4_0: R19.2, TP5.1, U3.5 (A4)
- new net A5_0: R20.2, TP6.1, U3.24 (A5)
- new net CH0_0: U3.6 (LED0)
- new net CH0_1: U3.7 (LED1)
- new net CH0_10: U3.17 (LED10)
- new net CH0_11: U3.18 (LED11)
- new net CH0_12: U3.19 (LED12)
- new net CH0_13: U3.20 (LED13)
- new net CH0_14: U3.21 (LED14)
- new net CH0_15: U3.22 (LED15)
- new net CH0_2: U3.8 (LED2)
- new net CH0_3: U3.9 (LED3)
- new net CH0_4: U3.10 (LED4)
- new net CH0_5: U3.11 (LED5)
- new net CH0_6: U3.12 (LED6)
- new net CH0_7: U3.13 (LED7)
- new net CH0_8: U3.15 (LED8)
- new net CH0_9: U3.16 (LED9)
- new net GND: C29.1, C30.1, R15.1, R16.1, R17.1, R18.1, R19.1, R20.1, R21.1, U3.14 (VSS), U3.25 (EXTCLK)
- new net PCA9685_I2C_SCL: U3.26 (SCL)
- new net PCA9685_I2C_SDA: U3.27 (SDA)
Other:
- title: (none) -> SERVO DRIVERS
