File: hardware/Source/Ver_1.1.0/ThermalFan.kicad_sch (KiCad schematic)
At the start: 0 parts

Commit message: Update Library for Ver 2
Parts:
- added J5: Connector, automative_hexapod:JST-XH-SMD-2-2.54mm, symbol automative_hexapod:JST-XH-SMD-2-2.54mm
- added Q5: LN2302LT1G, automative_hexapod:SOT23, symbol automative_hexapod:LN2302LT1G
- added R26: 4.7Ohm, automative_hexapod:Res_0603, symbol automative_hexapod:Res_4.7_0603_1%
- added R27: 10kOhm, automative_hexapod:Res_0603, symbol automative_hexapod:Res_10K_0603_1%
Connections:
- new net: Q5.1 (G), R26.2, R27.2
- new net BBAI_PWM1A: R26.1
- new net GND: Q5.2 (S), R27.1
Other:
- title: (none) -> THERMAL FAN
