File: hardware/Source/Ver_1.1.0/ConnectorServo.kicad_sch (KiCad schematic)
At the start: 54 parts, among them J10 Connector, J11 Connector, J12 Connector, J13 Connector, J14 Connector, J15 Connector, J16 Connector, J17 Connector, J18 Connector, J19 Connector, J20 Connector, J21 Connector, J22 Connector, J23 Connector, J24 Connector, J7 Connector, J8 Connector, J9 Connector

Commit message: update pcb and schematic
Parts:
- renumbered C39 to C33, C40 to C34, C41 to C35, C42 to C36, C43 to C37, C44 to C38, C45 to C39, C46 to C40, C47 to C41, C48 to C42, C49 to C43, C50 to C44, C51 to C45, C52 to C46, C53 to C47, C54 to C48, C55 to C49, C56 to C50, C57 to C51, C58 to C52, C59 to C53, C60 to C54, C61 to C55, C62 to C56, C63 to C57, C64 to C58, C65 to C59, C66 to C60, C67 to C61, C68 to C62, C69 to C63, C70 to C64, C71 to C65, C72 to C66, C73 to C67, C74 to C68
Connections:
- net GND: now also J10.SH (Pin_3), J11.SH (Pin_3), J12.SH (Pin_3), J13.SH (Pin_3), J14.SH (Pin_3), J15.SH (Pin_3), J16.SH (Pin_3), J17.SH (Pin_3), J18.SH (Pin_3), J19.SH (Pin_3), J20.SH (Pin_3), J21.SH (Pin_3), J22.SH (Pin_3), J23.SH (Pin_3), J24.SH (Pin_3), J7.SH (Pin_3), J8.SH (Pin_3), J9.SH (Pin_3)
- net Vdrive renamed Vdrive_1
- net Vdrive_1: no longer C33.2, C34.2, C35.2, C36.2, C37.2, C38.2, C39.2, C40.2, C41.2, C42.2, C43.2, C44.2, C45.2, C46.2, C47.2, C48.2, C49.2, C50.2, J10.2 (Pin_2), J11.2 (Pin_2), J12.2 (Pin_2), J13.2 (Pin_2), J14.2 (Pin_2), J15.2 (Pin_2), J7.2 (Pin_2), J8.2 (Pin_2), J9.2 (Pin_2)
- new net Vdrive_2: C33.2, C34.2, C35.2, C36.2, C37.2, C38.2, C39.2, C40.2, C41.2, C42.2, C43.2, C44.2, C45.2, C46.2, C47.2, C48.2, C49.2, C50.2, J10.2 (Pin_2), J11.2 (Pin_2), J12.2 (Pin_2), J13.2 (Pin_2), J14.2 (Pin_2), J15.2 (Pin_2), J7.2 (Pin_2), J8.2 (Pin_2), J9.2 (Pin_2)
Other:
- moved on the sheet: C36, C41, C43, C45, C46, C47, C49, C50, C61, C62, C63, C65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
